Commit message: launch file single for all hands, that launch also gazebo, heri files taken from this repo and heri real inertias added

File: configs/urdf/heri.urdf (robot description, URDF)
Before this commit: robot iit_heri_ros, 13 links, 12 joints
Joints:
- joint LFP1_1__LFP1_2: mimic (none) -> joint=LFB1__LFP1_1 multiplier=1 offset=0
- joint LFP1_2__LFP1_3: mimic (none) -> joint=LFB1__LFP1_1 multiplier=1 offset=0
- joint LFP2_1__LFP2_2: mimic (none) -> joint=LFB2__LFP2_1 multiplier=1 offset=0
- joint LFP2_2__LFP2_3: mimic (none) -> joint=LFB2__LFP2_1 multiplier=1 offset=0
- joint SFP1_1__SFP1_2: mimic (none) -> joint=SFB1__SFP1_1 multiplier=1 offset=0
