Commit message: damp and frictions very low so simulation works

File: configs/urdf/heri_real.urdf (robot description, URDF)
Before this commit: robot heri_real, 13 links, 12 joints
Joints:
- joint LFP1_1__LFP1_2: mimic (none) -> joint=LFB1__LFP1_1 multiplier=1 offset=0
- joint LFP2_1__LFP2_2: mimic (none) -> joint=LFB2_1__LFP2_1 multiplier=1 offset=0
- joint LFP2_2__LFP2_3: mimic (none) -> joint=LFB2__LFP2_1 multiplier=1 offset=0
- joint SFP1_1__SFP1_2: mimic (none) -> joint=SFB1__SFP1_1 multiplier=1 offset=0
- joint world_base: origin xyz=0 0 0.01 rpy=0 0 0 -> xyz=0 0 0.015 rpy=0 0 0

File: configs/urdf/heri_real.xacro (robot description, xacro)
@@ -9,5 +9,7 @@
   <link name="world"/>
   <joint name="world_base" type="fixed">
-    <origin xyz="0 0 0.01" rpy="0 0 0" />
+    <!-- z!= from 1 is necessary because otherwise the hand has tremors. I think this is because it compentetrate with the
+         terrain ? -->
+    <origin xyz="0 0 0.015" rpy="0 0 0" />
     <parent link="world" />
     <child link="base_link"/>
@@ -65,5 +67,5 @@
     <axis xyz="0 0 1" />
     <limit lower="-0.1" upper="0.1" effort="10" velocity="1" />
-    <dynamics damping="0.7" />
+    <dynamics damping="0.003" friction="0.003"/>
   </joint>
   <!-- ///////////////////////////////////////   First phalanx of the Short_Finger   ////////////////////////////////////////// -->
@@ -97,5 +99,5 @@
     <axis xyz="0 0 -1" />
     <limit lower="-0.1" upper="0.5" effort="10" velocity="1" />
-    <dynamics damping="0.7" />
+    <dynamics damping="0.003" friction="0.003"/>
   </joint>
   <!-- ///////////////////////////////////////   Tip phalanx of the short finger   ////////////////////////////////////////// -->
@@ -129,6 +131,10 @@
     <axis xyz="0 0 -1" />
     <limit lower="-0.1" upper="0.5" effort="10" velocity="1" />
-    <dynamics damping="0.7" />
-  </joint>
+    <dynamics damping="0.003" friction="0.003"/>
+    <mimic joint="SFB1__SFP1_1" multiplier="1" offset="0"/>
+  </joint>
+      <xacro:mimic_joint_plugin_gazebo name_prefix="SFP1_1__SFP1_2_joint"
+    parent_joint="SFB1__SFP1_1" mimic_joint="SFP1_1__SFP1_2"
+    has_pid="false" multiplier="1.0" max_effort="10.0" />
 <!-- ///////////////////////////////////////   Long finger 1   ////////////////////////////////////////// -->
   <!-- ///////////////////////////////////////   Base_Link of the long_finger   ////////////////////////////////////////// -->
@@ -162,5 +168,5 @@
     <axis xyz="0 0 1" />
     <limit lower="-0.1" upper="0.1" effort="10" velocity="1" />
-    <dynamics damping="0.7" />
+    <dynamics damping="0.003" friction="0.003"/>
   </joint>
   <!-- ///////////////////////////////////////   First phalanx of the Long_Finger   ////////////////////////////////////////// -->
@@ -194,5 +200,5 @@
     <axis xyz="0 0 -1" />
     <limit lower="-0.1" upper="0.5" effort="10" velocity="1" />
-    <dynamics damping="0.7" />
+    <dynamics damping="0.003" friction="0.003"/>
   </joint>
   <!-- ///////////////////////////////////////   Second phalanx of the Long_Finger   ////////////////////////////////////////// -->
@@ -226,6 +232,10 @@
     <axis xyz="0 0 -1" />
     <limit lower="-0.1" upper="0.5" effort="10" velocity="1" />
-    <dynamics damping="0.7" />
-  </joint>
+    <dynamics damping="0.003" friction="0.003"/>
+    <mimic joint="LFB1__LFP1_1" multiplier="1" offset="0"/>
+  </joint>
+        <xacro:mimic_joint_plugin_gazebo name_prefix="LFP1_1__LFP1_2_joint"
+    parent_joint="LFB1__LFP1_1" mimic_joint="LFP1_1__LFP1_2"
+    has_pid="false" multiplier="1.0" max_effort="10.0" />
   <!-- ///////////////////////////////////////   Tip phalanx of the long finger   ////////////////////////////////////////// -->
   <link name="LFP1_3">
@@ -258,6 +268,9 @@
     <axis xyz="0 0 -1" />
     <limit lower="-0.1" upper="0.5" effort="10" velocity="1" />
-    <dynamics damping="0.7" />
-  </joint>
+    <dynamics damping="0.003" friction="0.003"/>
+  </joint>
+        <xacro:mimic_joint_plugin_gazebo name_prefix="LFP1_1__LFP1_3_joint"
+    parent_joint="LFB1__LFP1_1" mimic_joint="LFP1_2__LFP1_3"
+    has_pid="false" multiplier="1.0" max_effort="10.0" />
   <!-- ///////////////////////////////////////   Long finger 2   ////////////////////////////////////////// -->
   <!-- ///////////////////////////////////////   Base_Link of the long_finger   ////////////////////////////////////////// -->
@@ -291,5 +304,5 @@
     <axis xyz="0 0 1" />
     <limit lower="-0.1" upper="0.1" effort="10" velocity="1" />
-    <dynamics damping="0.7" />
+    <dynamics damping="0.003" friction="0.003"/>
   </joint>
   <!-- ///////////////////////////////////////   First phalanx of the Long_Finger   ////////////////////////////////////////// -->
@@ -323,5 +336,5 @@
     <axis xyz="0 0 -1" />
     <limit lower="-0.1" upper="0.5" effort="10" velocity="1" />
-    <dynamics damping="0.7" />
+    <dynamics damping="0.003" friction="0.003"/>
   </joint>
   <!-- ///////////////////////////////////////   Second phalanx of the Long_Finger   ////////////////////////////////////////// -->
@@ -355,6 +368,10 @@
     <axis xyz="0 0 -1" />
     <limit lower="-0.1" upper="0.5" effort="10" velocity="1"/>
-    <dynamics damping="0.7" />
-  </joint>
+    <dynamics damping="0.003" friction="0.003"/>
+    <mimic joint="LFB2_1__LFP2_1" multiplier="1" offset="0"/>
+  </joint>
+          <xacro:mimic_joint_plugin_gazebo name_prefix="LFP2_1__LFP2_2_joint"
+    parent_joint="LFB2__LFP2_1" mimic_joint="LFP2_1__LFP2_2"
+    has_pid="false" multiplier="1.0" max_effort="10.0" />
   <!-- ///////////////////////////////////////   Tip phalanx of the long finger   ////////////////////////////////////////// -->
   <link name="LFP2_3">
@@ -387,5 +404,9 @@
     <axis xyz="0 0 -1" />
     <limit lower="-0.1" upper="0.5" effort="10" velocity="1"/>
-    <dynamics damping="0.7" />
-  </joint>
+    <dynamics damping="0.003" friction="0.003"/>
+    <mimic joint="LFB2__LFP2_1" multiplier="1" offset="0"/>
+  </joint>
+            <xacro:mimic_joint_plugin_gazebo name_prefix="LFP2_2__LFP2_3_joint"
+    parent_joint="LFB2__LFP2_1" mimic_joint="LFP2_2__LFP2_3"
+    has_pid="false" multiplier="1.0" max_effort="10.0" />
 </robot>
