Commit message: heri models corrected

File: configs/urdf/heri.xacro (robot description, xacro)
@@ -9,4 +9,6 @@
   <link name="world"/>
   <joint name="world_base" type="fixed">
+    <!-- z!= from 1 is necessary because otherwise the hand has tremors. I think this is because it compentetrate
+     with the terrain ? -->
     <origin xyz="0 0 0.015" rpy="0 0 0" />
     <parent link="world" />

File: configs/urdf/heri_real.urdf (robot description, URDF)
Before this commit: robot heri_real, 13 links, 12 joints
Joints:
- joint LFP1_2__LFP1_3: mimic (none) -> joint=LFB1__LFP1_1 multiplier=1 offset=0
- joint LFP2_1__LFP2_2: mimic joint=LFB2_1__LFP2_1 multiplier=1 offset=0 -> joint=LFB2__LFP2_1 multiplier=1 offset=0

File: configs/urdf/heri_real.xacro (robot description, xacro)
@@ -269,4 +269,5 @@
     <limit lower="-0.1" upper="0.5" effort="10" velocity="1" />
     <dynamics damping="0.003" friction="0.003"/>
+    <mimic joint="LFB1__LFP1_1" multiplier="1" offset="0"/>
   </joint>
         <xacro:mimic_joint_plugin_gazebo name_prefix="LFP1_1__LFP1_3_joint"
@@ -369,5 +370,5 @@
     <limit lower="-0.1" upper="0.5" effort="10" velocity="1"/>
     <dynamics damping="0.003" friction="0.003"/>
-    <mimic joint="LFB2_1__LFP2_1" multiplier="1" offset="0"/>
+    <mimic joint="LFB2__LFP2_1" multiplier="1" offset="0"/>
   </joint>
           <xacro:mimic_joint_plugin_gazebo name_prefix="LFP2_1__LFP2_2_joint"
