Commit message: added models and config for heri 4 fingers

File: configs/urdf/heri_II_real.urdf (robot description, URDF)
Before this commit: robot heri_real, 13 links, 12 joints
Links:
- added link LFB3, mass 0.0039598861; collision mesh filename=package://heri_description/meshes/LFB3.STL; visual mesh filename=package://heri_description/meshes/LFB3.STL
- added link LFP3_1, mass 0.021630428; collision mesh filename=package://heri_description/meshes/LFP3_1.STL; visual mesh filename=package://heri_description/meshes/LFP3_1.STL
- added link LFP3_2, mass 0.022869549; collision mesh filename=package://heri_description/meshes/LFP3_2.STL; visual mesh filename=package://heri_description/meshes/LFP3_2.STL
- added link LFP3_3, mass 0.02226615; collision mesh filename=package://heri_description/meshes/LFP3_3.STL; visual mesh filename=package://heri_description/meshes/LFP3_3.STL
- link LFB1: mass 4.1065000E-03 -> 0.0039598861
- link LFB2: mass 4.1065000E-03 -> 0.0039598861
- link LFP1_1: mass 2.1732283E-02 -> 0.021630428
- link LFP1_2: mass 2.2971404E-02 -> 0.022869549
- link LFP1_3: mass 2.2266150E-02 -> 0.02226615
- link LFP2_1: mass 2.1732283E-02 -> 0.021630428
- link LFP2_2: mass 2.2971404E-02 -> 0.022869549
- link LFP2_3: mass 2.2266150E-02 -> 0.02226615
- link SFB1_1: mass 2.1732283E-02 -> 0.021630428
- link SFP1_2: mass 2.2266150E-02 -> 0.02226615
- link base_link: geometry collision mesh filename=package://heri_description/meshes/base_link.STL; visual mesh filename=package://heri_description/meshes/base_heri_ii.STL
Joints:
- added joint BASE__LFB3: type revolute, parent base_link, child LFB3, origin xyz=0.030998 0.025903 0.1213 rpy=1.5708 -1.5708 3.1415927, axis 0 0 1, limit lower=-0.1 upper=0.1 effort=10 velocity=1
- added joint LFB3__LFP3_1: type revolute, parent LFB3, child LFP3_1, origin xyz=0.011 0 0.007 rpy=1.5708 -0.29671 0, axis 0 0 -1, limit lower=-0.1 upper=0.5 effort=10 velocity=1
- added joint LFP3_1__LFP3_2: type revolute, parent LFP3_1, child LFP3_2, origin xyz=0.035 0 0 rpy=0 0 0, axis 0 0 -1, limit lower=-0.1 upper=0.5 effort=10 velocity=1, mimic joint=LFB3__LFP3_1 multiplier=1 offset=0
- added joint LFP3_2__LFP3_3: type revolute, parent LFP3_2, child LFP3_3, origin xyz=0.035 0 0 rpy=0 0 0, axis 0 0 -1, limit lower=-0.1 upper=0.5 effort=10 velocity=1, mimic joint=LFB3__LFP3_1 multiplier=1 offset=0
- joint BASE__LFB1: origin xyz=-0.0167 0.0405 0.0635 rpy=1.5708 -1.5708 3.1415927 -> xyz=-0.031002 0.025903 0.1213 rpy=1.5708 -1.5708 3.1415927
- joint BASE__LFB2: origin xyz=0.0353 0.0405 0.0635 rpy=1.5708 -1.5708 3.1415927 -> xyz=0 0.031903 0.1213 rpy=1.5708 -1.5708 3.1415927
- joint BASE__SFB1: origin xyz=-0.0167 -0.0405 0.0635 rpy=1.5708 -1.5708 0 -> xyz=7.6421E-05 -0.031634 0.1213 rpy=1.5708 -1.5708 0

File: configs/urdf/heri_II_real.xacro (robot description, xacro)
@@ -1,4 +1,4 @@
 <?xml version="1.0" encoding="utf-8"?>
-<robot name="heri_real" xmlns:xacro="http://ros.org/wiki/xacro">
+<robot name="heri_II_real" xmlns:xacro="http://ros.org/wiki/xacro">
   <!-- Import all Gazebo-customization elements, including Gazebo colors -->
   <xacro:include filename="$(find ros_end_effector)/configs/urdf/iit_heri_ros.gazebo" />
@@ -24,5 +24,5 @@
       <origin xyz="0 0 0" rpy="0 0 0" />
       <geometry>
-        <mesh filename="package://heri_description/meshes/base_link.STL" />
+        <mesh filename="package://heri_description/meshes/base_heri_ii.STL" />
       </geometry>
       <material name="">
@@ -62,5 +62,5 @@
   <!-- ///////////////////////////////////////   Joint of BASE and the base_link of the short finger   ////////////////////////////////////////// -->
   <joint name="BASE__SFB1" type="revolute">
-    <origin xyz="-0.0167 -0.0405 0.0635" rpy="1.5708 -1.5708 0" />
+    <origin xyz="7.6421E-05 -0.031634 0.1213" rpy="1.5708 -1.5708 0" />
     <parent link="base_link" />
     <child link="SFB1" />
@@ -72,6 +72,6 @@
   <link name="SFB1_1">
     <inertial>
-      <origin xyz="1.3557103E-02 -1.5667663E-04 1.4446853E-04" rpy="0 0 0" />
-      <mass value="2.1732283E-02" />
+      <origin xyz="0.013537693 -0.00011389541 0.00014514898" rpy="0 0 0" />
+      <mass value="0.021630428" />
       <inertia ixx="1.7547572E-06" ixy="1.2425281E-07" ixz="-5.2776703E-08" iyy="7.3422819E-06" iyz="-1.1395559E-09" izz="7.1587820E-06" />
     </inertial>
@@ -104,6 +104,6 @@
   <link name="SFP1_2">
     <inertial>
-      <origin xyz="1.2398348E-02 -3.4958691E-04 5.0212619E-05" rpy="0 0 0" />
-      <mass value="2.2266150E-02" />
+      <origin xyz="0.012398348 -0.00034958691 0.000050212619" rpy="0 0 0" />
+      <mass value="0.02226615" />
       <inertia ixx="1.7400409E-06" ixy="4.4309075E-07" ixz="-1.3771833E-08" iyy="6.8917616E-06" iyz="6.4562527E-09" izz="6.4653229E-06" />
     </inertial>
@@ -141,6 +141,6 @@
   <link name="LFB1">
     <inertial>
-      <origin xyz="3.9400487E-03 0 6.4488006E-03" rpy="0 0 0" />
-      <mass value="4.1065000E-03" />
+      <origin xyz="0.000045491656 -0.0037522651 0.0064111226" rpy="0 0 0" />
+      <mass value="0.0039598861" />
       <inertia ixx="4.3061452E-07" ixy="0" ixz="-1.2027573E-07" iyy="3.9605806E-07" iyz="0" izz="3.9738552E-07" />
     </inertial>
@@ -163,5 +163,5 @@
   <!-- ///////////////////////////////////////   Joint of BASE and the base_link of the short finger   ////////////////////////////////////////// -->
   <joint name="BASE__LFB1" type="revolute">
-    <origin xyz="-0.0167 0.0405 0.0635" rpy="1.5708 -1.5708 3.1415927" />
+    <origin xyz="-0.031002 0.025903 0.1213" rpy="1.5708 -1.5708 3.1415927" />
     <parent link="base_link" />
     <child link="LFB1" />
@@ -173,6 +173,6 @@
   <link name="LFP1_1">
     <inertial>
-      <origin xyz="1.3557103E-02 -1.5667663E-04 1.4446853E-04" rpy="0 0 0" />
-      <mass value="2.1732283E-02" />
+      <origin xyz="0.013537693 -0.00011389541 0.00014514898" rpy="0 0 0" />
+      <mass value="0.021630428" />
       <inertia ixx="1.7547572E-06" ixy="1.2425281E-07" ixz="-5.2776703E-08" iyy="7.3422819E-06" iyz="-1.1395559E-09" izz="7.1587820E-06" />
     </inertial>
@@ -205,6 +205,6 @@
   <link name="LFP1_2">
     <inertial>
-      <origin xyz="1.2838417E-02 2.5385905E-04 1.2711003E-04" rpy="0 0 0" />
-      <mass value="2.2971404E-02" />
+      <origin xyz="0.012816858 0.00029615072 0.00012767631" rpy="0 0 0" />
+      <mass value="0.022869549" />
       <inertia ixx="1.9943688E-06" ixy="1.3380251E-07" ixz="-5.3468405E-08" iyy="7.4922799E-06" iyz="-9.2812315E-10" izz="7.3102836E-06" />
     </inertial>
@@ -232,5 +232,5 @@
     <axis xyz="0 0 -1" />
     <limit lower="-0.1" upper="0.5" effort="10" velocity="1" />
-    <dynamics damping="0.003" friction="0.003"/>
+    <dynamics damping="0.06" friction="0.05"/>
     <mimic joint="LFB1__LFP1_1" multiplier="1" offset="0"/>
   </joint>
@@ -241,6 +241,6 @@
   <link name="LFP1_3">
     <inertial>
-      <origin xyz="1.2398348E-02 -3.4958691E-04 5.0212619E-05" rpy="0 0 0" />
-      <mass value="2.2266150E-02" />
+      <origin xyz="0.012398348 -0.00034958691 0.000050212619" rpy="0 0 0" />
+      <mass value="0.02226615" />
       <inertia ixx="1.7400409E-06" ixy="4.4309075E-07" ixz="-1.3771833E-08" iyy="6.8917616E-06" iyz="6.4562527E-09" izz="6.4653229E-06" />
     </inertial>
@@ -278,6 +278,6 @@
   <link name="LFB2">
     <inertial>
-      <origin xyz="3.9400487E-03 0 6.4488006E-03" rpy="0 0 0" />
-      <mass value="4.1065000E-03" />
+      <origin xyz="0.000045491656 -0.0037522651 0.0064111226" rpy="0 0 0" />
+      <mass value="0.0039598861" />
       <inertia ixx="4.3061452E-07" ixy="0" ixz="-1.2027573E-07" iyy="3.9605806E-07" iyz="0" izz="3.9738552E-07" />
     </inertial>
@@ -300,5 +300,5 @@
   <!-- ///////////////////////////////////////   Joint of BASE and the base_link of the short finger   ////////////////////////////////////////// -->
   <joint name="BASE__LFB2" type="revolute">
-    <origin xyz="0.0353 0.0405 0.0635" rpy="1.5708 -1.5708 3.1415927" />
+    <origin xyz="0 0.031903 0.1213" rpy="1.5708 -1.5708 3.1415927" />
     <parent link="base_link" />
     <child link="LFB2" />
@@ -310,6 +310,6 @@
   <link name="LFP2_1">
     <inertial>
-      <origin xyz="1.3557103E-02 -1.5667663E-04 1.4446853E-04" rpy="0 0 0" />
-      <mass value="2.1732283E-02" />
+      <origin xyz="0.013537693 -0.00011389541 0.00014514898" rpy="0 0 0" />
+      <mass value="0.021630428" />
       <inertia ixx="1.7547572E-06" ixy="1.2425281E-07" ixz="-5.2776703E-08" iyy="7.3422819E-06" iyz="-1.1395559E-09" izz="7.1587820E-06" />
     </inertial>
@@ -342,6 +342,6 @@
   <link name="LFP2_2">
     <inertial>
-      <origin xyz="1.2838417E-02 2.5385905E-04 1.2711003E-04" rpy="0 0 0" />
-      <mass value="2.2971404E-02" />
+      <origin xyz="0.012816858 0.00029615072 0.00012767631" rpy="0 0 0" />
+      <mass value="0.022869549" />
       <inertia ixx="1.9943688E-06" ixy="1.3380251E-07" ixz="-5.3468405E-08" iyy="7.4922799E-06" iyz="-9.2812315E-10" izz="7.3102836E-06" />
     </inertial>
@@ -372,5 +372,5 @@
     <mimic joint="LFB2__LFP2_1" multiplier="1" offset="0"/>
   </joint>
-  <xacro:mimic_joint_plugin_gazebo name_prefix="LFP2_1__LFP2_2_joint"
+          <xacro:mimic_joint_plugin_gazebo name_prefix="LFP2_1__LFP2_2_joint"
     parent_joint="LFB2__LFP2_1" mimic_joint="LFP2_1__LFP2_2"
     has_pid="false" multiplier="1.0" max_effort="10.0" />
@@ -378,6 +378,6 @@
   <link name="LFP2_3">
     <inertial>
-      <origin xyz="1.2398348E-02 -3.4958691E-04 5.0212619E-05" rpy="0 0 0" />
-      <mass value="2.2266150E-02" />
+      <origin xyz="0.012398348 -0.00034958691 0.000050212619" rpy="0 0 0" />
+      <mass value="0.02226615" />
       <inertia ixx="1.7400409E-06" ixy="4.4309075E-07" ixz="-1.3771833E-08" iyy="6.8917616E-06" iyz="6.4562527E-09" izz="6.4653229E-06" />
     </inertial>
@@ -405,5 +405,5 @@
     <axis xyz="0 0 -1" />
     <limit lower="-0.1" upper="0.5" effort="10" velocity="1"/>
-    <dynamics damping="0.003" friction="0.003"/>
+    <dynamics damping="0.06" friction="0.05"/>
     <mimic joint="LFB2__LFP2_1" multiplier="1" offset="0"/>
   </joint>
@@ -411,6 +411,143 @@
     parent_joint="LFB2__LFP2_1" mimic_joint="LFP2_2__LFP2_3"
     has_pid="false" multiplier="1.0" max_effort="10.0" />
+  <!-- ///////////////////////////////////////   Long finger 3   ////////////////////////////////////////// -->
+  <!-- ///////////////////////////////////////   Base_Link of the long_finger   ////////////////////////////////////////// -->
+  <link name="LFB3">
+    <inertial>
+      <origin xyz="0.000045491656 -0.0037522651 0.0064111226" rpy="0 0 0" />
+      <mass value="0.0039598861" />
+      <inertia ixx="4.3061452E-07" ixy="0" ixz="-1.2027573E-07" iyy="3.9605806E-07" iyz="0" izz="3.9738552E-07" />
+    </inertial>
+    <visual>
+      <origin xyz="0 0 0" rpy="0 0 0" />
+      <geometry>
+        <mesh filename="package://heri_description/meshes/LFB3.STL" />
+      </geometry>
+      <material name="">
+        <color rgba="0.75294 0.75294 0.75294 1" />
+      </material>
+    </visual>
+    <collision>
+      <origin xyz="0 0 0" rpy="0 0 0" />
+      <geometry>
+        <mesh filename="package://heri_description/meshes/LFB3.STL" />
+      </geometry>
+    </collision>
+  </link>
+  <!-- ///////////////////////////////////////   Joint of BASE and the base_link of the short finger   ////////////////////////////////////////// -->
+  <joint name="BASE__LFB3" type="revolute">
+    <origin xyz="0.030998 0.025903 0.1213" rpy="1.5708 -1.5708 3.1415927" />
+    <parent link="base_link" />
+    <child link="LFB3" />
+    <axis xyz="0 0 1" />
+    <limit lower="-0.1" upper="0.1" effort="10" velocity="1" />
+    <dynamics damping="0.003" friction="0.003"/>
+  </joint>
+  <!-- ///////////////////////////////////////   First phalanx of the Long_Finger   ////////////////////////////////////////// -->
+  <link name="LFP3_1">
+    <inertial>
+      <origin xyz="0.013537693 -0.00011389541 0.00014514898" rpy="0 0 0" />
+      <mass value="0.021630428" />
+      <inertia ixx="1.7547572E-06" ixy="1.2425281E-07" ixz="-5.2776703E-08" iyy="7.3422819E-06" iyz="-1.1395559E-09" izz="7.1587820E-06" />
+    </inertial>
+    <visual>
+      <origin xyz="0 0 0" rpy="0 0 0" />
+      <geometry>
+        <mesh filename="package://heri_description/meshes/LFP3_1.STL" />
+      </geometry>
+      <material name="">
+        <color rgba="0.75294 0.75294 0.75294 1" />
+      </material>
+    </visual>
+    <collision>
+      <origin xyz="0 0 0" rpy="0 0 0" />
+      <geometry>
+        <mesh filename="package://heri_description/meshes/LFP3_1.STL" />
+      </geometry>
+    </collision>
+  </link>
+  <!-- ///////////////////////////////////////   Joint of base_link and the first phalanx of the short finger   ////////////////////////////////////////// -->
+  <joint name="LFB3__LFP3_1" type="revolute">
+    <origin xyz="0.011 0 0.007" rpy="1.5708 -0.29671 0" />
+    <parent link="LFB3" />
+    <child link="LFP3_1" />
+    <axis xyz="0 0 -1" />
+    <limit lower="-0.1" upper="0.5" effort="10" velocity="1" />
+    <dynamics damping="0.003" friction="0.003"/>
+  </joint>
+  <!-- ///////////////////////////////////////   Second phalanx of the Long_Finger   ////////////////////////////////////////// -->
+  <link name="LFP3_2">
+    <inertial>
+      <origin xyz="0.012816858 0.00029615072 0.00012767631" rpy="0 0 0" />
+      <mass value="0.022869549" />
+      <inertia ixx="1.9943688E-06" ixy="1.3380251E-07" ixz="-5.3468405E-08" iyy="7.4922799E-06" iyz="-9.2812315E-10" izz="7.3102836E-06" />
+    </inertial>
+    <visual>
+      <origin xyz="0 0 0" rpy="0 0 0" />
+      <geometry>
+        <mesh filename="package://heri_description/meshes/LFP3_2.STL" />
+      </geometry>
+      <material name="">
+        <color rgba="0.75294 0.75294 0.75294 1" />
+      </material>
+    </visual>
+    <collision>
+      <origin xyz="0 0 0" rpy="0 0 0" />
+      <geometry>
+        <mesh filename="package://heri_description/meshes/LFP3_2.STL" />
+      </geometry>
+    </collision>
+  </link>
+  <!-- ///////////////////////////////////////   Joint of base_link and the first phalanx of the short finger   ////////////////////////////////////////// -->
+  <joint name="LFP3_1__LFP3_2" type="revolute">
+    <origin xyz="0.035 0 0" rpy="0 0 0" />
+    <parent link="LFP3_1" />
+    <child link="LFP3_2" />
+    <axis xyz="0 0 -1" />
+    <limit lower="-0.1" upper="0.5" effort="10" velocity="1"/>
+    <dynamics damping="0.003" friction="0.003"/>
+    <mimic joint="LFB3__LFP3_1" multiplier="1" offset="0"/>
+  </joint>
+  <xacro:mimic_joint_plugin_gazebo name_prefix="LFP3_1__LFP3_2_joint"
+    parent_joint="LFB3__LFP3_1" mimic_joint="LFP3_1__LFP3_2"
+    has_pid="false" multiplier="1.0" max_effort="10.0" />
+  <!-- ///////////////////////////////////////   Tip phalanx of the long finger   ////////////////////////////////////////// -->
+  <link name="LFP3_3">
+    <inertial>
+      <origin xyz="0.012398348 -0.00034958691 0.000050212619" rpy="0 0 0" />
+      <mass value="0.02226615" />
+      <inertia ixx="1.7400409E-06" ixy="4.4309075E-07" ixz="-1.3771833E-08" iyy="6.8917616E-06" iyz="6.4562527E-09" izz="6.4653229E-06" />
+    </inertial>
+    <visual>
+      <origin xyz="0 0 0" rpy="0 0 0" />
+      <geometry>
+        <mesh filename="package://heri_description/meshes/LFP3_3.STL" />
+      </geometry>
+      <material name="">
+        <color rgba="0.75294 0.75294 0.75294 1" />
+      </material>
+    </visual>
+    <collision>
+      <origin xyz="0 0 0" rpy="0 0 0" />
+      <geometry>
+        <mesh filename="package://heri_description/meshes/LFP3_3.STL" />
+      </geometry>
+    </collision>
+  </link>
+  <!-- ///////////////////////////////////////   Joint of second and tip phalanxs of the long finger   ////////////////////////////////////////// -->
+  <joint name="LFP3_2__LFP3_3" type="revolute">
+    <origin xyz="0.035 0 0" rpy="0 0 0" />
+    <parent link="LFP3_2" />
+    <child link="LFP3_3" />
+    <axis xyz="0 0 -1" />
+    <limit lower="-0.1" upper="0.5" effort="10" velocity="1"/>
+    <dynamics damping="0.003" friction="0.003"/>
+    <mimic joint="LFB3__LFP3_1" multiplier="1" offset="0"/>
+  </joint>
+  <xacro:mimic_joint_plugin_gazebo name_prefix="LFP3_2__LFP3_3_joint"
+    parent_joint="LFB3__LFP3_1" mimic_joint="LFP3_2__LFP3_3"
+    has_pid="false" multiplier="1.0" max_effort="10.0" />
   <gazebo>
-    <plugin name="heri_real_controller" filename="libRoseePlugin.so">
+    <plugin name="heri_II_real_controller" filename="libRoseePlugin.so">
     </plugin>
   </gazebo>
