Commit message: event better mimic params

File: configs/urdf/heri_II_realLimits.urdf (robot description, URDF)
Before this commit: robot heri_II_realLimits, 17 links, 16 joints
Joints:
- joint LFP1_1__LFP1_2: mimic joint=LFB1__LFP1_1 multiplier=1 offset=0 -> joint=LFB1__LFP1_1 multiplier=1 offset=0.1
- joint LFP1_2__LFP1_3: mimic joint=LFB1__LFP1_1 multiplier=0.5 offset=0 -> joint=LFB1__LFP1_1 multiplier=0.5 offset=0.2
- joint LFP2_1__LFP2_2: mimic joint=LFB2__LFP2_1 multiplier=1 offset=0 -> joint=LFB2__LFP2_1 multiplier=1 offset=0.1
- joint LFP2_2__LFP2_3: mimic joint=LFB2__LFP2_1 multiplier=0.5 offset=0 -> joint=LFB2__LFP2_1 multiplier=0.5 offset=0.2
- joint LFP3_1__LFP3_2: mimic joint=LFB3__LFP3_1 multiplier=1 offset=0 -> joint=LFB3__LFP3_1 multiplier=1 offset=0.1
- joint LFP3_2__LFP3_3: mimic joint=LFB3__LFP3_1 multiplier=0.5 offset=0 -> joint=LFB3__LFP3_1 multiplier=0.5 offset=0.2
- joint SFP1_1__SFP1_2: mimic joint=SFB1__SFP1_1 multiplier=0.3 offset=0 -> joint=SFB1__SFP1_1 multiplier=0.3 offset=0.2
