Commit message: trying to use moto pos for dynamic model

File: configs/urdf/heri_II_current.urdf (robot description, URDF)
Before this commit: robot heri_II, 17 links, 16 joints
Joints:
- joint BASE__LFB1: type revolute -> fixed
- joint BASE__LFB2: type revolute -> fixed
- joint BASE__LFB3: type revolute -> fixed
- joint BASE__SFB1: type revolute -> fixed
- joint LFP1_1__LFP1_2: limit lower=-0.1 upper=0.5 effort=10 velocity=1 -> lower=-0.1 upper=1.1 effort=10 velocity=1
- joint LFP1_2__LFP1_3: limit lower=-0.1 upper=0.5 effort=10 velocity=1 -> lower=-0.1 upper=1.1 effort=10 velocity=1
