Commit message: add/improved config and launch files for robotiq-3f

File: configs/urdf/robotiq_3f.urdf (robot description, URDF)
Before this commit: robot robotiq-3f-gripper_articulated, 14 links, 13 joints
Links:
- added link base_link
Joints:
- added joint base_link_to_palm: type fixed, parent base_link, child palm, origin xyz=0 0 0 rpy=1.57079632679 0 0

Commit message: updated robotiq-3f for gazebo simul

File: configs/urdf/robotiq_3f.urdf (robot description, URDF)
Before this commit: robot robotiq_3f, 15 links, 14 joints
Links:
- added link world
- link palm: mass None -> 1.3
Joints:
- added joint virtualFixed: type fixed, parent world, child base_link
- joint finger_1_joint_2: mimic (none) -> joint=finger_1_joint_1 multiplier=0.85 offset=0
- joint finger_1_joint_3: mimic (none) -> joint=finger_1_joint_1 multiplier=0.8 offset=0
- joint finger_2_joint_2: mimic (none) -> joint=finger_2_joint_1 multiplier=0.85 offset=0
- joint finger_2_joint_3: mimic (none) -> joint=finger_2_joint_1 multiplier=0.8 offset=0
- joint finger_middle_joint_2: mimic (none) -> joint=finger_middle_joint_1 multiplier=0.85 offset=0
- joint finger_middle_joint_3: mimic (none) -> joint=finger_middle_joint_1 multiplier=0.8 offset=0

Commit message: updated robotiq model

File: configs/urdf/robotiq_3f.urdf (robot description, URDF)
Before this commit: robot robotiq_3f, 16 links, 15 joints
Links:
- removed link base_link
Joints:
- removed joint base_link_to_palm
- removed joint virtualFixed
- added joint world_base: type fixed, parent world, child palm, origin xyz=0 0 0 rpy=1.57079632679 0 0
