Commit message: corrected HERI 2 model

File: configs/urdf/heri_II.xacro (robot description, xacro)
@@ -94,5 +94,5 @@
   <!-- ///////////////////////////////////////   Joint of base_link and the first phalanx of the short finger   ////////////////////////////////////////// -->
   <joint name="SFB1__SFP1_1" type="revolute">
-    <origin xyz="0.011 0 0.007" rpy="1.5708 -0.29671 0" />
+		<origin xyz="0.0211 0 0.007" rpy="1.5708 -0.29671 0" />
     <parent link="SFB1" />
     <child link="SFB1_1" />

File: configs/urdf/heri_II_current.urdf (robot description, URDF)
Before this commit: robot heri_II, 17 links, 16 joints
Joints:
- joint SFB1__SFP1_1: origin xyz=0.011 0 0.007 rpy=1.5708 -0.29671 0 -> xyz=0.0211 0 0.007 rpy=1.5708 -0.29671 0

File: configs/urdf/heri_II_new.urdf (robot description, URDF)
Before this commit: robot heri_II_new, 21 links, 20 joints
Joints:
- joint SFB1__SFP1_1: origin xyz=0.011 0 0.007 rpy=1.5708 -0.29671 0 -> xyz=0.0211 0 0.007 rpy=1.5708 -0.29671 0

Commit message: Corrected thumb frame

File: configs/urdf/heri_II.xacro (robot description, xacro)
@@ -94,5 +94,5 @@
   <!-- ///////////////////////////////////////   Joint of base_link and the first phalanx of the short finger   ////////////////////////////////////////// -->
   <joint name="SFB1__SFP1_1" type="revolute">
-		<origin xyz="0.0211 0 0.007" rpy="1.5708 -0.29671 0" />
+    <origin xyz="0.0256 0 0.007" rpy="1.5708 -0.29671 0" />
     <parent link="SFB1" />
     <child link="SFB1_1" />

Commit message: Revert "Corrected thumb frame"
This reverts commit 0e6720302c7230b037e3872a19783845a2e78ecd.

going back to right x value in urdf for heri thumb

File: configs/urdf/heri_II.xacro (robot description, xacro)
@@ -94,5 +94,5 @@
   <!-- ///////////////////////////////////////   Joint of base_link and the first phalanx of the short finger   ////////////////////////////////////////// -->
   <joint name="SFB1__SFP1_1" type="revolute">
-    <origin xyz="0.0256 0 0.007" rpy="1.5708 -0.29671 0" />
+		<origin xyz="0.0211 0 0.007" rpy="1.5708 -0.29671 0" />
     <parent link="SFB1" />
     <child link="SFB1_1" />
