Commit message: organized heri urdf files

File: configs/urdf/heri_II_NL.urdf (robot description, URDF)
Before this commit: robot heri_II_NL, 21 links, 20 joints
Links:
- link motor_finger1_virtual_link: mass None -> 0.01
- link motor_finger2_virtual_link: mass None -> 0.01
- link motor_finger3_virtual_link: mass None -> 0.01
- link motor_thumb_virtual_link: mass None -> 0.01
Joints:
- joint SFB1__SFP1_1: origin xyz=0.011 0 0.007 rpy=1.5708 -0.29671 0 -> xyz=0.0211 0 0.007 rpy=1.5708 -0.29671 0

File: configs/urdf/heri_II_NL.xacro (robot description, xacro)
@@ -99,9 +99,33 @@
     </collision>
   </link>
-   <!-- I Put motors as joints, linked to tree with virtual links  -->
-  <link name="motor_finger1_virtual_link" />
-  <link name="motor_finger2_virtual_link" />
-  <link name="motor_finger3_virtual_link" />
-  <link name="motor_thumb_virtual_link" />
+  <!-- I Put motors as joints, linked to tree with virtual links  -->
+  <link name="motor_finger1_virtual_link">
+   <inertial> <!-- We need inertial otherwise gazebo does not load the motor joints. I put very low inertia-->
+      <origin rpy="0 0 0" xyz="0 0 0"/>
+      <mass value="0.01"/>
+      <inertia ixx="0.0001" ixy="0.0" ixz="0.0" iyy="0.0001" iyz="0.0" izz="0.0001"/>
+    </inertial>
+  </link>
+  <link name="motor_finger2_virtual_link">
+   <inertial> <!-- We need inertial otherwise gazebo does not load the motor joints. I put very low inertia-->
+      <origin rpy="0 0 0" xyz="0 0 0"/>
+      <mass value="0.01"/>
+      <inertia ixx="0.0001" ixy="0.0" ixz="0.0" iyy="0.0001" iyz="0.0" izz="0.0001"/>
+    </inertial>
+  </link>
+  <link name="motor_finger3_virtual_link">
+     <inertial> <!-- We need inertial otherwise gazebo does not load the motor joints. I put very low inertia-->
+      <origin rpy="0 0 0" xyz="0 0 0"/>
+      <mass value="0.01"/>
+      <inertia ixx="0.0001" ixy="0.0" ixz="0.0" iyy="0.0001" iyz="0.0" izz="0.0001"/>
+    </inertial>
+  </link>
+  <link name="motor_thumb_virtual_link">
+     <inertial> <!-- We need inertial otherwise gazebo does not load the motor joints. I put very low inertia-->
+      <origin rpy="0 0 0" xyz="0 0 0"/>
+      <mass value="0.01"/>
+      <inertia ixx="0.0001" ixy="0.0" ixz="0.0" iyy="0.0001" iyz="0.0" izz="0.0001"/>
+    </inertial>
+  </link>
   <joint name="motor_finger1" type="revolute">
     <origin rpy="0 0 0" xyz="0 0 0"/>
@@ -189,5 +213,5 @@
   <!-- ///////////////////////////////////////   Joint of base_link and the first phalanx of the short finger   ////////////////////////////////////////// -->
   <joint name="SFB1__SFP1_1" type="revolute">
-    <origin xyz="0.011 0 0.007" rpy="1.5708 -0.29671 0" />
+    <origin xyz="0.0211 0 0.007" rpy="1.5708 -0.29671 0" />
     <parent link="SFB1" />
     <child link="SFB1_1" />

Commit message: corrected non linear heri rel

File: configs/urdf/heri_II_NL.urdf (robot description, URDF)
Before this commit: robot heri_II_NL, 21 links, 20 joints
Joints:
- joint LFB1__LFP1_1: limit lower=-0.1 upper=0.9 effort=10 velocity=1 -> lower=-0.1 upper=0.56 effort=10 velocity=1
- joint LFB2__LFP2_1: limit lower=-0.1 upper=0.73 effort=10 velocity=1 -> lower=-0.1 upper=0.56 effort=10 velocity=1
- joint LFB3__LFP3_1: limit lower=-0.1 upper=0.9 effort=10 velocity=1 -> lower=-0.1 upper=0.56 effort=10 velocity=1
- joint LFP1_1__LFP1_2: limit lower=-0.1 upper=0.5 effort=10 velocity=1 -> lower=-0.1 upper=1.22 effort=10 velocity=1
- joint LFP1_2__LFP1_3: limit lower=-0.1 upper=0.5 effort=10 velocity=1 -> lower=-0.1 upper=1.22 effort=10 velocity=1
- joint LFP2_1__LFP2_2: limit lower=-0.1 upper=0.5 effort=10 velocity=1 -> lower=-0.1 upper=1.22 effort=10 velocity=1
- joint LFP2_2__LFP2_3: limit lower=-0.1 upper=0.5 effort=10 velocity=1 -> lower=-0.1 upper=1.22 effort=10 velocity=1
- joint LFP3_1__LFP3_2: limit lower=-0.1 upper=0.5 effort=10 velocity=1 -> lower=-0.1 upper=1.22 effort=10 velocity=1
- joint LFP3_2__LFP3_3: limit lower=-0.1 upper=0.5 effort=10 velocity=1 -> lower=-0.1 upper=1.22 effort=10 velocity=1
- joint SFB1__SFP1_1: limit lower=-0.1 upper=0.9 effort=10 velocity=1 -> lower=-0.1 upper=1.22 effort=10 velocity=1
- joint SFP1_1__SFP1_2: limit lower=-0.1 upper=1.2 effort=10 velocity=1 -> lower=-0.1 upper=1.22 effort=10 velocity=1

File: configs/urdf/heri_II_NL.xacro (robot description, xacro)
@@ -1,18 +1,13 @@
 <?xml version="1.0" encoding="utf-8"?>
 <robot name="heri_II_NL" xmlns:xacro="http://ros.org/wiki/xacro">
+	<xacro:property name="exp" value="2.71828" />
     <!-- macro to for non linear functions, that are the same for each fingers-->
   <xacro:macro name="mimic_non_linear_long_finger" params="father_joint phalange regression_level:=high">
   	<xacro:if value="${phalange == 'proximal'}">    <!-- joint of the first phalange -->
-			<xacro:if value="${regression_level == 'low'}">
-				<xacro:property name="p" value="${[0.7528, -0.9162, 0.7495, 0.0005927]}"/>
-				<mimic joint="${father_joint}" nlFunPos="${p[0]}*x^3 + ${p[1]}*x^2 + ${p[2]}*x + ${p[3]}"/>
-			</xacro:if>
-			<xacro:if value="${regression_level == 'medium'}">
-				<xacro:property name="p" value="${[-0.506, 1.698, -1.453, 0.8461, -0.002379 ]}"/>
-				<mimic joint="${father_joint}" nlFunPos="${p[0]}*x^4 + ${p[1]}*x^3 + ${p[2]}*x^2 + ${p[3]}*x + ${p[4]}"/>
-			</xacro:if>
 			<xacro:if value="${regression_level == 'high'}">
-				<xacro:property name="p" value="${[-3.986, 8.428, -5.14, 0.6392, 0.6254, 0.001261]}"/>
-				<mimic joint="${father_joint}" nlFunPos="${p[0]}*x^5 + ${p[1]}*x^4 + ${p[2]}*x^3 + ${p[3]}*x^2 + ${p[4]}*x + ${p[5]}"/>
+				<xacro:property name="a" value="${[0.08519, 21500000000000, -714900,  0.2555]}"/>
+				<xacro:property name="b" value="${[0.9172,  32.2,           -17.93,   0.7317]}"/>
+				<xacro:property name="c" value="${[0.1817,  5.513,          4.61,     1.105]}"/>
+				<mimic joint="${father_joint}" nlFunPos="${a[0]}*${exp}^(-((x-${b[0]})/${c[0]})^2) + ${a[1]}*${exp}^(-((x-${b[1]})/${c[1]})^2) + ${a[2]}*${exp}^(-((x-${b[2]})/${c[2]})^2) + ${a[3]}*${exp}^(-((x-${b[3]})/${c[3]})^2)"/>
 			</xacro:if>
     </xacro:if>
@@ -27,5 +22,5 @@
 			</xacro:if>
 			<xacro:if value="${regression_level == 'high'}">
-				<xacro:property name="p" value="${[0.1099, -0.6142, 0.4386, 0.658,  0.0009892]}"/>
+				<xacro:property name="p" value="${[-0.1028, 0.4311, -0.6019, 0.9364,  -0.01132]}"/>
 				<mimic joint="${father_joint}" nlFunPos="${p[0]}*x^4 + ${p[1]}*x^3 + ${p[2]}*x^2 +${p[3]}*x + ${p[4]}"/>
 			</xacro:if>
@@ -41,6 +36,6 @@
 			</xacro:if>
 			<xacro:if value="${regression_level == 'high'}">
-				<xacro:property name="p" value="${[0.08032, -0.216, -0.07007, 0.5351, 0.000428]}"/>
-				<mimic joint="${father_joint}" nlFunPos="${p[0]}*x^4 + ${p[1]}*x^3 + ${p[2]}*x^2 +${p[3]}*x + ${p[4]}"/>
+				<xacro:property name="p" value="${[-0.06965, 0.4258, -0.7659, 0.3528, 0.4078, 0.007414]}"/>
+				<mimic joint="${father_joint}" nlFunPos="${p[0]}*x^5 + ${p[1]}*x^4 + ${p[2]}*x^3 +${p[3]}*x^2 + ${p[4]}*x + ${p[5]}"/>
 			</xacro:if>
     </xacro:if>
@@ -53,5 +48,5 @@
 				</xacro:if>
 				<xacro:if value="${regression_level == 'high'}">
-  				<xacro:property name="p" value="${[-9.144, 11.02, -3.932, 1.401, -0.002157]}"/>
+  				<xacro:property name="p" value="${[0.3378, -1.179, 1.103, 0.7363, 0.01468]}"/>
 					<mimic joint="${father_joint}" nlFunPos="${p[0]}*x^4 + ${p[1]}*x^3 + ${p[2]}*x^2 + ${p[3]}*x + ${p[4]}"/>
 				</xacro:if>
@@ -63,5 +58,5 @@
 				</xacro:if>
 				<xacro:if value="${regression_level == 'high'}">
-  				<xacro:property name="p" value="${[6.076, -7.902, 2.248, 0.739, 0.001644]}"/>
+  				<xacro:property name="p" value="${[-0.3366, 1.674, -2.506, 1.552, -0.02812]}"/>
 					<mimic joint="${father_joint}" nlFunPos="${p[0]}*x^4 + ${p[1]}*x^3 + ${p[2]}*x^2 + ${p[3]}*x + ${p[4]}"/>
 				</xacro:if>
@@ -198,5 +193,5 @@
     <child link="SFB1_1" />
     <axis xyz="0 0 -1" />
-    <limit lower="-0.1" upper="0.9" effort="10" velocity="1" />
+    <limit lower="-0.1" upper="1.22" effort="10" velocity="1" />
     <dynamics damping="0.003" friction="0.003"/>
     <xacro:mimic_non_linear_short_finger father_joint="motor_thumb" phalange="proximal" />
@@ -231,5 +226,5 @@
     <child link="SFP1_2" />
     <axis xyz="0 0 -1" />
-    <limit lower="-0.1" upper="1.2" effort="10" velocity="1" />
+    <limit lower="-0.1" upper="1.22" effort="10" velocity="1" />
     <dynamics damping="0.003" friction="0.003"/>
     <xacro:mimic_non_linear_short_finger father_joint="motor_thumb" phalange="distal" />
@@ -297,5 +292,5 @@
     <child link="LFP1_1" />
     <axis xyz="0 0 -1" />
-    <limit lower="-0.1" upper="0.9" effort="10" velocity="1" />
+    <limit lower="-0.1" upper="0.56" effort="10" velocity="1" />
     <dynamics damping="0.003" friction="0.003"/>
     <xacro:mimic_non_linear_long_finger father_joint="motor_finger1" phalange="proximal" />
@@ -330,5 +325,5 @@
     <child link="LFP1_2" />
     <axis xyz="0 0 -1" />
-    <limit lower="-0.1" upper="0.5" effort="10" velocity="1" />
+    <limit lower="-0.1" upper="1.22" effort="10" velocity="1" />
     <dynamics damping="0.06" friction="0.05"/>
     <xacro:mimic_non_linear_long_finger father_joint="motor_finger1" phalange="middle" />
@@ -363,5 +358,5 @@
     <child link="LFP1_3" />
     <axis xyz="0 0 -1" />
-    <limit lower="-0.1" upper="0.5" effort="10" velocity="1" />
+    <limit lower="-0.1" upper="1.22" effort="10" velocity="1" />
     <dynamics damping="0.003" friction="0.003"/>
     <xacro:mimic_non_linear_long_finger father_joint="motor_finger1" phalange="distal" />
@@ -429,5 +424,5 @@
     <child link="LFP2_1" />
     <axis xyz="0 0 -1" />
-    <limit lower="-0.1" upper="0.73" effort="10" velocity="1" />
+    <limit lower="-0.1" upper="0.56" effort="10" velocity="1" />
     <dynamics damping="0.003" friction="0.003"/>
     <xacro:mimic_non_linear_long_finger father_joint="motor_finger2" phalange="proximal" />
@@ -462,5 +457,5 @@
     <child link="LFP2_2" />
     <axis xyz="0 0 -1" />
-    <limit lower="-0.1" upper="0.5" effort="10" velocity="1"/>
+    <limit lower="-0.1" upper="1.22" effort="10" velocity="1"/>
     <dynamics damping="0.003" friction="0.003"/>
     <xacro:mimic_non_linear_long_finger father_joint="motor_finger2" phalange="middle" />
@@ -495,5 +490,5 @@
     <child link="LFP2_3" />
     <axis xyz="0 0 -1" />
-    <limit lower="-0.1" upper="0.5" effort="10" velocity="1"/>
+    <limit lower="-0.1" upper="1.22" effort="10" velocity="1"/>
     <dynamics damping="0.06" friction="0.05"/>
     <xacro:mimic_non_linear_long_finger father_joint="motor_finger2" phalange="distal" />
@@ -561,5 +556,5 @@
     <child link="LFP3_1" />
     <axis xyz="0 0 -1" />
-    <limit lower="-0.1" upper="0.9" effort="10" velocity="1" />
+    <limit lower="-0.1" upper="0.56" effort="10" velocity="1" />
     <dynamics damping="0.003" friction="0.003"/>
     <xacro:mimic_non_linear_long_finger father_joint="motor_finger3" phalange="proximal" />
@@ -594,5 +589,5 @@
     <child link="LFP3_2" />
     <axis xyz="0 0 -1" />
-    <limit lower="-0.1" upper="0.5" effort="10" velocity="1"/>
+    <limit lower="-0.1" upper="1.22" effort="10" velocity="1"/>
     <dynamics damping="0.003" friction="0.003"/>
     <xacro:mimic_non_linear_long_finger father_joint="motor_finger3" phalange="middle" />
@@ -627,5 +622,5 @@
     <child link="LFP3_3" />
     <axis xyz="0 0 -1" />
-    <limit lower="-0.1" upper="0.5" effort="10" velocity="1"/>
+    <limit lower="-0.1" upper="1.22" effort="10" velocity="1"/>
     <dynamics damping="0.003" friction="0.003"/>
     <xacro:mimic_non_linear_long_finger father_joint="motor_finger3" phalange="distal" />

Commit message: added virtual link on fingertips border

File: configs/urdf/heri_II_NL.urdf (robot description, URDF)
Before this commit: robot heri_II_NL, 21 links, 20 joints
Links:
- added link LFP1_3_tip, mass 0.01
- added link LFP2_3_tip, mass 0.01
- added link LFP3_3_tip, mass 0.01
- added link SFP1_2_tip, mass 0.01
Joints:
- added joint LFP1_3__LFP1_3_tip: type fixed, parent LFP1_3, child LFP1_3_tip, origin xyz=0.0175 -0.0111 0 rpy=1.5708 0 -0.13, axis 0 0 0
- added joint LFP2_3__LFP2_3_tip: type fixed, parent LFP2_3, child LFP2_3_tip, origin xyz=0.0175 -0.0111 0 rpy=1.5708 0 -0.13, axis 0 0 0
- added joint LFP3_3__LFP3_3_tip: type fixed, parent LFP3_3, child LFP3_3_tip, origin xyz=0.0175 -0.0111 0 rpy=1.5708 0 -0.13, axis 0 0 0
- added joint SFP1_2__SFP1_2_tip: type fixed, parent SFP1_2, child SFP1_2_tip, origin xyz=0.0175 -0.0111 0 rpy=1.5708 0 -0.13, axis 0 0 0

File: configs/urdf/heri_II_NL.xacro (robot description, xacro)
@@ -650,3 +650,56 @@
     <xacro:mimic_non_linear_long_finger father_joint="motor_finger3" phalange="distal" />
   </joint>
+  <!-- //////////////////////////////////////////// virtual links to put a frame on fingertip "skin" //////////////////////////////////////////-->
+  <link name="LFP3_3_tip">
+   <inertial> <!-- We need inertial otherwise gazebo does not load the motor joints. I put very low inertia-->
+      <origin rpy="0 0 0" xyz="0 0 0"/>
+      <mass value="0.01"/>
+      <inertia ixx="0.0001" ixy="0.0" ixz="0.0" iyy="0.0001" iyz="0.0" izz="0.0001"/>
+    </inertial>
+  </link>
+  <joint name="LFP3_3__LFP3_3_tip" type="fixed">
+    <origin rpy="1.5708 0 -0.13" xyz="0.0175 -0.0111 0"/>
+    <parent link="LFP3_3"/>
+    <child link="LFP3_3_tip"/>
+    <axis xyz="0 0 0"/>
+  </joint>
+  <link name="LFP2_3_tip">
+   <inertial> <!-- We need inertial otherwise gazebo does not load the motor joints. I put very low inertia-->
+      <origin rpy="0 0 0" xyz="0 0 0"/>
+      <mass value="0.01"/>
+      <inertia ixx="0.0001" ixy="0.0" ixz="0.0" iyy="0.0001" iyz="0.0" izz="0.0001"/>
+    </inertial>
+  </link>
+  <joint name="LFP2_3__LFP2_3_tip" type="fixed">
+    <origin rpy="1.5708 0 -0.13" xyz="0.0175 -0.0111 0"/>
+    <parent link="LFP2_3"/>
+    <child link="LFP2_3_tip"/>
+    <axis xyz="0 0 0"/>
+  </joint>
+  <link name="LFP1_3_tip">
+   <inertial> <!-- We need inertial otherwise gazebo does not load the motor joints. I put very low inertia-->
+      <origin rpy="0 0 0" xyz="0 0 0"/>
+      <mass value="0.01"/>
+      <inertia ixx="0.0001" ixy="0.0" ixz="0.0" iyy="0.0001" iyz="0.0" izz="0.0001"/>
+    </inertial>
+  </link>
+  <joint name="LFP1_3__LFP1_3_tip" type="fixed">
+    <origin rpy="1.5708 0 -0.13" xyz="0.0175 -0.0111 0"/>
+    <parent link="LFP1_3"/>
+    <child link="LFP1_3_tip"/>
+    <axis xyz="0 0 0"/>
+  </joint>
+  <link name="SFP1_2_tip">
+   <inertial> <!-- We need inertial otherwise gazebo does not load the motor joints. I put very low inertia-->
+      <origin rpy="0 0 0" xyz="0 0 0"/>
+      <mass value="0.01"/>
+      <inertia ixx="0.0001" ixy="0.0" ixz="0.0" iyy="0.0001" iyz="0.0" izz="0.0001"/>
+    </inertial>
+  </link>
+  <joint name="SFP1_2__SFP1_2_tip" type="fixed">
+    <origin rpy="1.5708 0 -0.13" xyz="0.0175 -0.0111 0"/>
+    <parent link="SFP1_2"/>
+    <child link="SFP1_2_tip"/>
+    <axis xyz="0 0 0"/>
+  </joint>
 </robot>
