Commit message: add meshes for heri II, renamed heri II files, deleted heri III files

File: configs/urdf/heri_II.urdf (robot description, URDF)
Before this commit: robot heri_real, 13 links, 12 joints
Links:
- added link LFB3, mass 0.0039598861; collision mesh filename=package://ros_end_effector/configs/meshes/heri_II/LFB3.STL; visual mesh filename=package://ros_end_effector/configs/meshes/heri_II/LFB3.STL
- added link LFP3_1, mass 0.021630428; collision mesh filename=package://ros_end_effector/configs/meshes/heri_II/LFP3_1.STL; visual mesh filename=package://ros_end_effector/configs/meshes/heri_II/LFP3_1.STL
- added link LFP3_2, mass 0.022869549; collision mesh filename=package://ros_end_effector/configs/meshes/heri_II/LFP3_2.STL; visual mesh filename=package://ros_end_effector/configs/meshes/heri_II/LFP3_2.STL
- added link LFP3_3, mass 0.02226615; collision mesh filename=package://ros_end_effector/configs/meshes/heri_II/LFP3_3.STL; visual mesh filename=package://ros_end_effector/configs/meshes/heri_II/LFP3_3.STL
- link LFB1: mass 4.1065000E-03 -> 0.0039598861; geometry collision mesh filename=package://ros_end_effector/configs/meshes/heri_II/LFB1.STL; visual mesh filename=package://ros_end_effector/configs/meshes/heri_II/LFB1.STL
- link LFB2: mass 4.1065000E-03 -> 0.0039598861; geometry collision mesh filename=package://ros_end_effector/configs/meshes/heri_II/LFB2.STL; visual mesh filename=package://ros_end_effector/configs/meshes/heri_II/LFB2.STL
- link LFP1_1: mass 2.1732283E-02 -> 0.021630428; geometry collision mesh filename=package://ros_end_effector/configs/meshes/heri_II/LFP1_1.STL; visual mesh filename=package://ros_end_effector/configs/meshes/heri_II/LFP1_1.STL
- link LFP1_2: mass 2.2971404E-02 -> 0.022869549; geometry collision mesh filename=package://ros_end_effector/configs/meshes/heri_II/LFP1_2.STL; visual mesh filename=package://ros_end_effector/configs/meshes/heri_II/LFP1_2.STL
- link LFP1_3: mass 2.2266150E-02 -> 0.02226615; geometry collision mesh filename=package://ros_end_effector/configs/meshes/heri_II/LFP1_3.STL; visual mesh filename=package://ros_end_effector/configs/meshes/heri_II/LFP1_3.STL
- link LFP2_1: mass 2.1732283E-02 -> 0.021630428; geometry collision mesh filename=package://ros_end_effector/configs/meshes/heri_II/LFP2_1.STL; visual mesh filename=package://ros_end_effector/configs/meshes/heri_II/LFP2_1.STL
- link LFP2_2: mass 2.2971404E-02 -> 0.022869549; geometry collision mesh filename=package://ros_end_effector/configs/meshes/heri_II/LFP2_2.STL; visual mesh filename=package://ros_end_effector/configs/meshes/heri_II/LFP2_2.STL
- link LFP2_3: mass 2.2266150E-02 -> 0.02226615; geometry collision mesh filename=package://ros_end_effector/configs/meshes/heri_II/LFP2_3.STL; visual mesh filename=package://ros_end_effector/configs/meshes/heri_II/LFP2_3.STL
- link SFB1: geometry collision mesh filename=package://ros_end_effector/configs/meshes/heri_II/SFB1.STL; visual mesh filename=package://ros_end_effector/configs/meshes/heri_II/SFB1.STL
- link SFB1_1: mass 2.1732283E-02 -> 0.021630428; geometry collision mesh filename=package://ros_end_effector/configs/meshes/heri_II/SFB1_1.STL; visual mesh filename=package://ros_end_effector/configs/meshes/heri_II/SFB1_1.STL
- link SFP1_2: mass 2.2266150E-02 -> 0.02226615; geometry collision mesh filename=package://ros_end_effector/configs/meshes/heri_II/SFP1_2.STL; visual mesh filename=package://ros_end_effector/configs/meshes/heri_II/SFP1_2.STL
- link base_link: geometry collision mesh filename=package://ros_end_effector/configs/meshes/heri_II/base_heri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; visual mesh filename=package://ros_end_effector/configs/meshes/heri_II/base_heri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
Joints:
- added joint BASE__LFB3: type revolute, parent base_link, child LFB3, origin xyz=0.030998 0.025903 0.1213 rpy=1.5708 -1.5708 3.1415927, axis 0 0 1, limit lower=-0.1 upper=0.1 effort=10 velocity=1
- added joint LFB3__LFP3_1: type revolute, parent LFB3, child LFP3_1, origin xyz=0.011 0 0.007 rpy=1.5708 -0.29671 0, axis 0 0 -1, limit lower=-0.1 upper=0.5 effort=10 velocity=1
- added joint LFP3_1__LFP3_2: type revolute, parent LFP3_1, child LFP3_2, origin xyz=0.035 0 0 rpy=0 0 0, axis 0 0 -1, limit lower=-0.1 upper=0.5 effort=10 velocity=1, mimic joint=LFB3__LFP3_1 multiplier=1 offset=0
- added joint LFP3_2__LFP3_3: type revolute, parent LFP3_2, child LFP3_3, origin xyz=0.035 0 0 rpy=0 0 0, axis 0 0 -1, limit lower=-0.1 upper=0.5 effort=10 velocity=1, mimic joint=LFB3__LFP3_1 multiplier=1 offset=0
- joint BASE__LFB1: origin xyz=-0.0167 0.0405 0.0635 rpy=1.5708 -1.5708 3.1415927 -> xyz=-0.031002 0.025903 0.1213 rpy=1.5708 -1.5708 3.1415927
- joint BASE__LFB2: origin xyz=0.0353 0.0405 0.0635 rpy=1.5708 -1.5708 3.1415927 -> xyz=0 0.031903 0.1213 rpy=1.5708 -1.5708 3.1415927
- joint BASE__SFB1: origin xyz=-0.0167 -0.0405 0.0635 rpy=1.5708 -1.5708 0 -> xyz=7.6421E-05 -0.031634 0.1213 rpy=1.5708 -1.5708 0

File: configs/urdf/heri_II.xacro (robot description, xacro)
@@ -1,8 +1,8 @@
 <?xml version="1.0" encoding="utf-8"?>
-<robot name="heri_II_real" xmlns:xacro="http://ros.org/wiki/xacro">
+<robot name="heri_II" xmlns:xacro="http://ros.org/wiki/xacro">
   <!-- Import all Gazebo-customization elements, including Gazebo colors -->
   <xacro:include filename="$(find ros_end_effector)/configs/urdf/iit_heri_ros.gazebo" />
   <!-- Import Rviz colors -->
-  <xacro:include filename="$(find heri_description)/urdf/materials.xacro" />
+  <xacro:include filename="$(find ros_end_effector)/configs/urdf/materials.xacro" />
   <!-- ///////////////////////////////////////   Short Finger   ////////////////////////////////////////// -->
   <!-- ///////////////////////////////////////   base_link   ////////////////////////////////////////// -->
@@ -24,14 +24,14 @@
       <origin xyz="0 0 0" rpy="0 0 0" />
       <geometry>
-        <mesh filename="package://heri_description/meshes/base_heri_ii.STL" />
-      </geometry>
-      <material name="">
-        <color rgba="0.75294 0.75294 0.75294 1" />
-      </material>
-    </visual>
-    <collision>
-      <origin xyz="0 0 0" rpy="0 0 0" />
-      <geometry>
-        <mesh filename="package://heri_description/meshes/base_link.STL" />
+        <mesh filename="package://ros_end_effector/configs/meshes/heri_II/base_heri_ii.STL" />
+      </geometry>
+      <material name="">
+        <color rgba="0.75294 0.75294 0.75294 1" />
+      </material>
+    </visual>
+    <collision>
+      <origin xyz="0 0 0" rpy="0 0 0" />
+      <geometry>
+        <mesh filename="package://ros_end_effector/configs/meshes/heri_II/base_heri_ii.STL" />
       </geometry>
     </collision>
@@ -47,14 +47,14 @@
       <origin xyz="0 0 0" rpy="0 0 0" />
       <geometry>
-        <mesh filename="package://heri_description/meshes/SFB1.STL" />
-      </geometry>
-      <material name="">
-        <color rgba="0.75294 0.75294 0.75294 1" />
-      </material>
-    </visual>
-    <collision>
-      <origin xyz="0 0 0" rpy="0 0 0" />
-      <geometry>
-        <mesh filename="package://heri_description/meshes/SFB1.STL" />
+        <mesh filename="package://ros_end_effector/configs/meshes/heri_II/SFB1.STL" />
+      </geometry>
+      <material name="">
+        <color rgba="0.75294 0.75294 0.75294 1" />
+      </material>
+    </visual>
+    <collision>
+      <origin xyz="0 0 0" rpy="0 0 0" />
+      <geometry>
+        <mesh filename="package://ros_end_effector/configs/meshes/heri_II/SFB1.STL" />
       </geometry>
     </collision>
@@ -79,14 +79,14 @@
       <origin xyz="0 0 0" rpy="0 0 0" />
       <geometry>
-        <mesh filename="package://heri_description/meshes/SFB1_1.STL" />
-      </geometry>
-      <material name="">
-        <color rgba="0.75294 0.75294 0.75294 1" />
-      </material>
-    </visual>
-    <collision>
-      <origin xyz="0 0 0" rpy="0 0 0" />
-      <geometry>
-        <mesh filename="package://heri_description/meshes/SFB1_1.STL" />
+        <mesh filename="package://ros_end_effector/configs/meshes/heri_II/SFB1_1.STL" />
+      </geometry>
+      <material name="">
+        <color rgba="0.75294 0.75294 0.75294 1" />
+      </material>
+    </visual>
+    <collision>
+      <origin xyz="0 0 0" rpy="0 0 0" />
+      <geometry>
+        <mesh filename="package://ros_end_effector/configs/meshes/heri_II/SFB1_1.STL" />
       </geometry>
     </collision>
@@ -111,14 +111,14 @@
       <origin xyz="0 0 0" rpy="0 0 0" />
       <geometry>
-        <mesh filename="package://heri_description/meshes/SFP1_2.STL" />
-      </geometry>
-      <material name="">
-        <color rgba="0.75294 0.75294 0.75294 1" />
-      </material>
-    </visual>
-    <collision>
-      <origin xyz="0 0 0" rpy="0 0 0" />
-      <geometry>
-        <mesh filename="package://heri_description/meshes/SFP1_2.STL" />
+        <mesh filename="package://ros_end_effector/configs/meshes/heri_II/SFP1_2.STL" />
+      </geometry>
+      <material name="">
+        <color rgba="0.75294 0.75294 0.75294 1" />
+      </material>
+    </visual>
+    <collision>
+      <origin xyz="0 0 0" rpy="0 0 0" />
+      <geometry>
+        <mesh filename="package://ros_end_effector/configs/meshes/heri_II/SFP1_2.STL" />
       </geometry>
     </collision>
@@ -148,14 +148,14 @@
       <origin xyz="0 0 0" rpy="0 0 0" />
       <geometry>
-        <mesh filename="package://heri_description/meshes/LFB1.STL" />
-      </geometry>
-      <material name="">
-        <color rgba="0.75294 0.75294 0.75294 1" />
-      </material>
-    </visual>
-    <collision>
-      <origin xyz="0 0 0" rpy="0 0 0" />
-      <geometry>
-        <mesh filename="package://heri_description/meshes/LFB1.STL" />
+        <mesh filename="package://ros_end_effector/configs/meshes/heri_II/LFB1.STL" />
+      </geometry>
+      <material name="">
+        <color rgba="0.75294 0.75294 0.75294 1" />
+      </material>
+    </visual>
+    <collision>
+      <origin xyz="0 0 0" rpy="0 0 0" />
+      <geometry>
+        <mesh filename="package://ros_end_effector/configs/meshes/heri_II/LFB1.STL" />
       </geometry>
     </collision>
@@ -180,14 +180,14 @@
       <origin xyz="0 0 0" rpy="0 0 0" />
       <geometry>
-        <mesh filename="package://heri_description/meshes/LFP1_1.STL" />
-      </geometry>
-      <material name="">
-        <color rgba="0.75294 0.75294 0.75294 1" />
-      </material>
-    </visual>
-    <collision>
-      <origin xyz="0 0 0" rpy="0 0 0" />
-      <geometry>
-        <mesh filename="package://heri_description/meshes/LFP1_1.STL" />
+        <mesh filename="package://ros_end_effector/configs/meshes/heri_II/LFP1_1.STL" />
+      </geometry>
+      <material name="">
+        <color rgba="0.75294 0.75294 0.75294 1" />
+      </material>
+    </visual>
+    <collision>
+      <origin xyz="0 0 0" rpy="0 0 0" />
+      <geometry>
+        <mesh filename="package://ros_end_effector/configs/meshes/heri_II/LFP1_1.STL" />
       </geometry>
     </collision>
@@ -212,14 +212,14 @@
       <origin xyz="0 0 0" rpy="0 0 0" />
       <geometry>
-        <mesh filename="package://heri_description/meshes/LFP1_2.STL" />
-      </geometry>
-      <material name="">
-        <color rgba="0.75294 0.75294 0.75294 1" />
-      </material>
-    </visual>
-    <collision>
-      <origin xyz="0 0 0" rpy="0 0 0" />
-      <geometry>
-        <mesh filename="package://heri_description/meshes/LFP1_2.STL" />
+        <mesh filename="package://ros_end_effector/configs/meshes/heri_II/LFP1_2.STL" />
+      </geometry>
+      <material name="">
+        <color rgba="0.75294 0.75294 0.75294 1" />
+      </material>
+    </visual>
+    <collision>
+      <origin xyz="0 0 0" rpy="0 0 0" />
+      <geometry>
+        <mesh filename="package://ros_end_effector/configs/meshes/heri_II/LFP1_2.STL" />
       </geometry>
     </collision>
@@ -248,14 +248,14 @@
       <origin xyz="0 0 0" rpy="0 0 0" />
       <geometry>
-        <mesh filename="package://heri_description/meshes/LFP1_3.STL" />
-      </geometry>
-      <material name="">
-        <color rgba="0.75294 0.75294 0.75294 1" />
-      </material>
-    </visual>
-    <collision>
-      <origin xyz="0 0 0" rpy="0 0 0" />
-      <geometry>
-        <mesh filename="package://heri_description/meshes/LFP1_3.STL" />
+        <mesh filename="package://ros_end_effector/configs/meshes/heri_II/LFP1_3.STL" />
+      </geometry>
+      <material name="">
+        <color rgba="0.75294 0.75294 0.75294 1" />
+      </material>
+    </visual>
+    <collision>
+      <origin xyz="0 0 0" rpy="0 0 0" />
+      <geometry>
+        <mesh filename="package://ros_end_effector/configs/meshes/heri_II/LFP1_3.STL" />
       </geometry>
     </collision>
@@ -285,14 +285,14 @@
       <origin xyz="0 0 0" rpy="0 0 0" />
       <geometry>
-        <mesh filename="package://heri_description/meshes/LFB2.STL" />
-      </geometry>
-      <material name="">
-        <color rgba="0.75294 0.75294 0.75294 1" />
-      </material>
-    </visual>
-    <collision>
-      <origin xyz="0 0 0" rpy="0 0 0" />
-      <geometry>
-        <mesh filename="package://heri_description/meshes/LFB2.STL" />
+        <mesh filename="package://ros_end_effector/configs/meshes/heri_II/LFB2.STL" />
+      </geometry>
+      <material name="">
+        <color rgba="0.75294 0.75294 0.75294 1" />
+      </material>
+    </visual>
+    <collision>
+      <origin xyz="0 0 0" rpy="0 0 0" />
+      <geometry>
+        <mesh filename="package://ros_end_effector/configs/meshes/heri_II/LFB2.STL" />
       </geometry>
     </collision>
@@ -317,14 +317,14 @@
       <origin xyz="0 0 0" rpy="0 0 0" />
       <geometry>
-        <mesh filename="package://heri_description/meshes/LFP2_1.STL" />
-      </geometry>
-      <material name="">
-        <color rgba="0.75294 0.75294 0.75294 1" />
-      </material>
-    </visual>
-    <collision>
-      <origin xyz="0 0 0" rpy="0 0 0" />
-      <geometry>
-        <mesh filename="package://heri_description/meshes/LFP2_1.STL" />
+        <mesh filename="package://ros_end_effector/configs/meshes/heri_II/LFP2_1.STL" />
+      </geometry>
+      <material name="">
+        <color rgba="0.75294 0.75294 0.75294 1" />
+      </material>
+    </visual>
+    <collision>
+      <origin xyz="0 0 0" rpy="0 0 0" />
+      <geometry>
+        <mesh filename="package://ros_end_effector/configs/meshes/heri_II/LFP2_1.STL" />
       </geometry>
     </collision>
@@ -349,14 +349,14 @@
       <origin xyz="0 0 0" rpy="0 0 0" />
       <geometry>
-        <mesh filename="package://heri_description/meshes/LFP2_2.STL" />
-      </geometry>
-      <material name="">
-        <color rgba="0.75294 0.75294 0.75294 1" />
-      </material>
-    </visual>
-    <collision>
-      <origin xyz="0 0 0" rpy="0 0 0" />
-      <geometry>
-        <mesh filename="package://heri_description/meshes/LFP2_2.STL" />
+        <mesh filename="package://ros_end_effector/configs/meshes/heri_II/LFP2_2.STL" />
+      </geometry>
+      <material name="">
+        <color rgba="0.75294 0.75294 0.75294 1" />
+      </material>
+    </visual>
+    <collision>
+      <origin xyz="0 0 0" rpy="0 0 0" />
+      <geometry>
+        <mesh filename="package://ros_end_effector/configs/meshes/heri_II/LFP2_2.STL" />
       </geometry>
     </collision>
@@ -385,14 +385,14 @@
       <origin xyz="0 0 0" rpy="0 0 0" />
       <geometry>
-        <mesh filename="package://heri_description/meshes/LFP2_3.STL" />
-      </geometry>
-      <material name="">
-        <color rgba="0.75294 0.75294 0.75294 1" />
-      </material>
-    </visual>
-    <collision>
-      <origin xyz="0 0 0" rpy="0 0 0" />
-      <geometry>
-        <mesh filename="package://heri_description/meshes/LFP2_3.STL" />
+        <mesh filename="package://ros_end_effector/configs/meshes/heri_II/LFP2_3.STL" />
+      </geometry>
+      <material name="">
+        <color rgba="0.75294 0.75294 0.75294 1" />
+      </material>
+    </visual>
+    <collision>
+      <origin xyz="0 0 0" rpy="0 0 0" />
+      <geometry>
+        <mesh filename="package://ros_end_effector/configs/meshes/heri_II/LFP2_3.STL" />
       </geometry>
     </collision>
@@ -422,14 +422,14 @@
       <origin xyz="0 0 0" rpy="0 0 0" />
       <geometry>
-        <mesh filename="package://heri_description/meshes/LFB3.STL" />
-      </geometry>
-      <material name="">
-        <color rgba="0.75294 0.75294 0.75294 1" />
-      </material>
-    </visual>
-    <collision>
-      <origin xyz="0 0 0" rpy="0 0 0" />
-      <geometry>
-        <mesh filename="package://heri_description/meshes/LFB3.STL" />
+        <mesh filename="package://ros_end_effector/configs/meshes/heri_II/LFB3.STL" />
+      </geometry>
+      <material name="">
+        <color rgba="0.75294 0.75294 0.75294 1" />
+      </material>
+    </visual>
+    <collision>
+      <origin xyz="0 0 0" rpy="0 0 0" />
+      <geometry>
+        <mesh filename="package://ros_end_effector/configs/meshes/heri_II/LFB3.STL" />
       </geometry>
     </collision>
@@ -454,14 +454,14 @@
       <origin xyz="0 0 0" rpy="0 0 0" />
       <geometry>
-        <mesh filename="package://heri_description/meshes/LFP3_1.STL" />
-      </geometry>
-      <material name="">
-        <color rgba="0.75294 0.75294 0.75294 1" />
-      </material>
-    </visual>
-    <collision>
-      <origin xyz="0 0 0" rpy="0 0 0" />
-      <geometry>
-        <mesh filename="package://heri_description/meshes/LFP3_1.STL" />
+        <mesh filename="package://ros_end_effector/configs/meshes/heri_II/LFP3_1.STL" />
+      </geometry>
+      <material name="">
+        <color rgba="0.75294 0.75294 0.75294 1" />
+      </material>
+    </visual>
+    <collision>
+      <origin xyz="0 0 0" rpy="0 0 0" />
+      <geometry>
+        <mesh filename="package://ros_end_effector/configs/meshes/heri_II/LFP3_1.STL" />
       </geometry>
     </collision>
@@ -486,14 +486,14 @@
       <origin xyz="0 0 0" rpy="0 0 0" />
       <geometry>
-        <mesh filename="package://heri_description/meshes/LFP3_2.STL" />
-      </geometry>
-      <material name="">
-        <color rgba="0.75294 0.75294 0.75294 1" />
-      </material>
-    </visual>
-    <collision>
-      <origin xyz="0 0 0" rpy="0 0 0" />
-      <geometry>
-        <mesh filename="package://heri_description/meshes/LFP3_2.STL" />
+        <mesh filename="package://ros_end_effector/configs/meshes/heri_II/LFP3_2.STL" />
+      </geometry>
+      <material name="">
+        <color rgba="0.75294 0.75294 0.75294 1" />
+      </material>
+    </visual>
+    <collision>
+      <origin xyz="0 0 0" rpy="0 0 0" />
+      <geometry>
+        <mesh filename="package://ros_end_effector/configs/meshes/heri_II/LFP3_2.STL" />
       </geometry>
     </collision>
@@ -522,14 +522,14 @@
       <origin xyz="0 0 0" rpy="0 0 0" />
       <geometry>
-        <mesh filename="package://heri_description/meshes/LFP3_3.STL" />
-      </geometry>
-      <material name="">
-        <color rgba="0.75294 0.75294 0.75294 1" />
-      </material>
-    </visual>
-    <collision>
-      <origin xyz="0 0 0" rpy="0 0 0" />
-      <geometry>
-        <mesh filename="package://heri_description/meshes/LFP3_3.STL" />
+        <mesh filename="package://ros_end_effector/configs/meshes/heri_II/LFP3_3.STL" />
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