Commit message: updated heri limits and mimic param in the normal file

File: configs/urdf/heri_II.urdf (robot description, URDF)
Before this commit: robot heri_II, 17 links, 16 joints
Joints:
- joint LFB1__LFP1_1: limit lower=-0.1 upper=0.5 effort=10 velocity=1 -> lower=-0.1 upper=0.9 effort=10 velocity=1
- joint LFB2__LFP2_1: limit lower=-0.1 upper=0.5 effort=10 velocity=1 -> lower=-0.1 upper=0.73 effort=10 velocity=1
- joint LFB3__LFP3_1: limit lower=-0.1 upper=0.5 effort=10 velocity=1 -> lower=-0.1 upper=0.9 effort=10 velocity=1
- joint LFP1_1__LFP1_2: mimic joint=LFB1__LFP1_1 multiplier=1 offset=0 -> joint=LFB1__LFP1_1 multiplier=1 offset=0.1
- joint LFP1_2__LFP1_3: mimic joint=LFB1__LFP1_1 multiplier=1 offset=0 -> joint=LFB1__LFP1_1 multiplier=0.5 offset=0.2
- joint LFP2_1__LFP2_2: mimic joint=LFB2__LFP2_1 multiplier=1 offset=0 -> joint=LFB2__LFP2_1 multiplier=1 offset=0.1
- joint LFP2_2__LFP2_3: mimic joint=LFB2__LFP2_1 multiplier=1 offset=0 -> joint=LFB2__LFP2_1 multiplier=0.5 offset=0.2
- joint LFP3_1__LFP3_2: mimic joint=LFB3__LFP3_1 multiplier=1 offset=0 -> joint=LFB3__LFP3_1 multiplier=1 offset=0.1
- joint LFP3_2__LFP3_3: mimic joint=LFB3__LFP3_1 multiplier=1 offset=0 -> joint=LFB3__LFP3_1 multiplier=0.5 offset=0.2
- joint SFB1__SFP1_1: limit lower=-0.1 upper=0.5 effort=10 velocity=1 -> lower=-0.1 upper=1.3 effort=10 velocity=1
- joint SFP1_1__SFP1_2: mimic joint=SFB1__SFP1_1 multiplier=1 offset=0 -> joint=SFB1__SFP1_1 multiplier=0.3 offset=0.2

File: configs/urdf/heri_II.xacro (robot description, xacro)
@@ -98,5 +98,5 @@
     <child link="SFB1_1" />
     <axis xyz="0 0 -1" />
-    <limit lower="-0.1" upper="0.5" effort="10" velocity="1" />
+    <limit lower="-0.1" upper="1.3" effort="10" velocity="1" />
     <dynamics damping="0.003" friction="0.003"/>
   </joint>
@@ -132,9 +132,9 @@
     <limit lower="-0.1" upper="0.5" effort="10" velocity="1" />
     <dynamics damping="0.003" friction="0.003"/>
-    <mimic joint="SFB1__SFP1_1" multiplier="1" offset="0"/>
+    <mimic joint="SFB1__SFP1_1" multiplier="0.3" offset="0.2"/>
   </joint>
       <xacro:mimic_joint_plugin_gazebo name_prefix="SFP1_1__SFP1_2_joint"
     parent_joint="SFB1__SFP1_1" mimic_joint="SFP1_1__SFP1_2"
-    has_pid="false" multiplier="1.0" max_effort="10.0" />
+    has_pid="false" multiplier="0.3" max_effort="10.0" offset="0.2"/>
 <!-- ///////////////////////////////////////   Long finger 1   ////////////////////////////////////////// -->
   <!-- ///////////////////////////////////////   Base_Link of the long_finger   ////////////////////////////////////////// -->
@@ -199,5 +199,5 @@
     <child link="LFP1_1" />
     <axis xyz="0 0 -1" />
-    <limit lower="-0.1" upper="0.5" effort="10" velocity="1" />
+    <limit lower="-0.1" upper="0.9" effort="10" velocity="1" />
     <dynamics damping="0.003" friction="0.003"/>
   </joint>
@@ -225,5 +225,5 @@
     </collision>
   </link>
-  <!-- ///////////////////////////////////////   Joint of base_link and the first phalanx of the short finger   ////////////////////////////////////////// -->
+  <!-- ///////////////////////////////////////   Joint of base_link and the first phalanx of the long finger   ////////////////////////////////////////// -->
   <joint name="LFP1_1__LFP1_2" type="revolute">
     <origin xyz="0.035 0 0" rpy="0 0 0" />
@@ -233,9 +233,9 @@
     <limit lower="-0.1" upper="0.5" effort="10" velocity="1" />
     <dynamics damping="0.06" friction="0.05"/>
-    <mimic joint="LFB1__LFP1_1" multiplier="1" offset="0"/>
+    <mimic joint="LFB1__LFP1_1" multiplier="1" offset="0.1"/>
   </joint>
         <xacro:mimic_joint_plugin_gazebo name_prefix="LFP1_1__LFP1_2_joint"
     parent_joint="LFB1__LFP1_1" mimic_joint="LFP1_1__LFP1_2"
-    has_pid="false" multiplier="1.0" max_effort="10.0" />
+    has_pid="false" multiplier="1.0" max_effort="10.0" offset="0.1" />
   <!-- ///////////////////////////////////////   Tip phalanx of the long finger   ////////////////////////////////////////// -->
   <link name="LFP1_3">
@@ -269,9 +269,9 @@
     <limit lower="-0.1" upper="0.5" effort="10" velocity="1" />
     <dynamics damping="0.003" friction="0.003"/>
-    <mimic joint="LFB1__LFP1_1" multiplier="1" offset="0"/>
+    <mimic joint="LFB1__LFP1_1" multiplier="0.5" offset="0.2"/>
   </joint>
         <xacro:mimic_joint_plugin_gazebo name_prefix="LFP1_1__LFP1_3_joint"
     parent_joint="LFB1__LFP1_1" mimic_joint="LFP1_2__LFP1_3"
-    has_pid="false" multiplier="1.0" max_effort="10.0" />
+    has_pid="false" multiplier="0.5" max_effort="10.0" offset="0.2" />
   <!-- ///////////////////////////////////////   Long finger 2   ////////////////////////////////////////// -->
   <!-- ///////////////////////////////////////   Base_Link of the long_finger   ////////////////////////////////////////// -->
@@ -336,5 +336,5 @@
     <child link="LFP2_1" />
     <axis xyz="0 0 -1" />
-    <limit lower="-0.1" upper="0.5" effort="10" velocity="1" />
+    <limit lower="-0.1" upper="0.73" effort="10" velocity="1" />
     <dynamics damping="0.003" friction="0.003"/>
   </joint>
@@ -370,9 +370,9 @@
     <limit lower="-0.1" upper="0.5" effort="10" velocity="1"/>
     <dynamics damping="0.003" friction="0.003"/>
-    <mimic joint="LFB2__LFP2_1" multiplier="1" offset="0"/>
+    <mimic joint="LFB2__LFP2_1" multiplier="1" offset="0.1"/>
   </joint>
           <xacro:mimic_joint_plugin_gazebo name_prefix="LFP2_1__LFP2_2_joint"
     parent_joint="LFB2__LFP2_1" mimic_joint="LFP2_1__LFP2_2"
-    has_pid="false" multiplier="1.0" max_effort="10.0" />
+    has_pid="false" multiplier="1.0" max_effort="10.0" offset="0.1" />
   <!-- ///////////////////////////////////////   Tip phalanx of the long finger   ////////////////////////////////////////// -->
   <link name="LFP2_3">
@@ -406,9 +406,9 @@
     <limit lower="-0.1" upper="0.5" effort="10" velocity="1"/>
     <dynamics damping="0.06" friction="0.05"/>
-    <mimic joint="LFB2__LFP2_1" multiplier="1" offset="0"/>
+    <mimic joint="LFB2__LFP2_1" multiplier="0.5" offset="0.2"/>
   </joint>
   <xacro:mimic_joint_plugin_gazebo name_prefix="LFP2_2__LFP2_3_joint"
     parent_joint="LFB2__LFP2_1" mimic_joint="LFP2_2__LFP2_3"
-    has_pid="false" multiplier="1.0" max_effort="10.0" />
+    has_pid="false" multiplier="0.5" max_effort="10.0" offset="0.2" />
   <!-- ///////////////////////////////////////   Long finger 3   ////////////////////////////////////////// -->
   <!-- ///////////////////////////////////////   Base_Link of the long_finger   ////////////////////////////////////////// -->
@@ -473,5 +473,5 @@
     <child link="LFP3_1" />
     <axis xyz="0 0 -1" />
-    <limit lower="-0.1" upper="0.5" effort="10" velocity="1" />
+    <limit lower="-0.1" upper="0.9" effort="10" velocity="1" />
     <dynamics damping="0.003" friction="0.003"/>
   </joint>
@@ -507,9 +507,9 @@
     <limit lower="-0.1" upper="0.5" effort="10" velocity="1"/>
     <dynamics damping="0.003" friction="0.003"/>
-    <mimic joint="LFB3__LFP3_1" multiplier="1" offset="0"/>
+    <mimic joint="LFB3__LFP3_1" multiplier="1" offset="0.1"/>
   </joint>
   <xacro:mimic_joint_plugin_gazebo name_prefix="LFP3_1__LFP3_2_joint"
     parent_joint="LFB3__LFP3_1" mimic_joint="LFP3_1__LFP3_2"
-    has_pid="false" multiplier="1.0" max_effort="10.0" />
+    has_pid="false" multiplier="1.0" max_effort="10.0" offset="0.1" />
   <!-- ///////////////////////////////////////   Tip phalanx of the long finger   ////////////////////////////////////////// -->
   <link name="LFP3_3">
@@ -543,8 +543,8 @@
     <limit lower="-0.1" upper="0.5" effort="10" velocity="1"/>
     <dynamics damping="0.003" friction="0.003"/>
-    <mimic joint="LFB3__LFP3_1" multiplier="1" offset="0"/>
+    <mimic joint="LFB3__LFP3_1" multiplier="0.5" offset="0.2"/>
   </joint>
   <xacro:mimic_joint_plugin_gazebo name_prefix="LFP3_2__LFP3_3_joint"
     parent_joint="LFB3__LFP3_1" mimic_joint="LFP3_2__LFP3_3"
-    has_pid="false" multiplier="1.0" max_effort="10.0" />
+    has_pid="false" multiplier="0.5" max_effort="10.0" offset="0.2"/>
 </robot>

Commit message: updated model param urdf/xacro

File: configs/urdf/heri_II.urdf (robot description, URDF)
Before this commit: robot heri_II, 17 links, 16 joints
Joints:
- joint SFB1__SFP1_1: limit lower=-0.1 upper=1.3 effort=10 velocity=1 -> lower=-0.1 upper=0.9 effort=10 velocity=1
- joint SFP1_1__SFP1_2: limit lower=-0.1 upper=0.5 effort=10 velocity=1 -> lower=-0.1 upper=1.2 effort=10 velocity=1; mimic joint=SFB1__SFP1_1 multiplier=0.3 offset=0.2 -> joint=SFB1__SFP1_1 multiplier=1.2 offset=0.2

File: configs/urdf/heri_II.xacro (robot description, xacro)
@@ -98,5 +98,5 @@
     <child link="SFB1_1" />
     <axis xyz="0 0 -1" />
-    <limit lower="-0.1" upper="1.3" effort="10" velocity="1" />
+    <limit lower="-0.1" upper="0.9" effort="10" velocity="1" />
     <dynamics damping="0.003" friction="0.003"/>
   </joint>
@@ -130,11 +130,11 @@
     <child link="SFP1_2" />
     <axis xyz="0 0 -1" />
-    <limit lower="-0.1" upper="0.5" effort="10" velocity="1" />
-    <dynamics damping="0.003" friction="0.003"/>
-    <mimic joint="SFB1__SFP1_1" multiplier="0.3" offset="0.2"/>
+    <limit lower="-0.1" upper="1.2" effort="10" velocity="1" />
+    <dynamics damping="0.003" friction="0.003"/>
+    <mimic joint="SFB1__SFP1_1" multiplier="1.2" offset="0.2"/>
   </joint>
       <xacro:mimic_joint_plugin_gazebo name_prefix="SFP1_1__SFP1_2_joint"
     parent_joint="SFB1__SFP1_1" mimic_joint="SFP1_1__SFP1_2"
-    has_pid="false" multiplier="0.3" max_effort="10.0" offset="0.2"/>
+    has_pid="false" multiplier="1.2" max_effort="10.0" offset="0.2"/>
 <!-- ///////////////////////////////////////   Long finger 1   ////////////////////////////////////////// -->
   <!-- ///////////////////////////////////////   Base_Link of the long_finger   ////////////////////////////////////////// -->

Commit message: lowered joint limit for thumb

File: configs/urdf/heri_II.urdf (robot description, URDF)
Before this commit: robot heri_II, 17 links, 16 joints
Joints:
- joint SFB1__SFP1_1: limit lower=-0.1 upper=0.9 effort=10 velocity=1 -> lower=-0.1 upper=0.2 effort=10 velocity=1
- joint SFP1_1__SFP1_2: mimic joint=SFB1__SFP1_1 multiplier=1.2 offset=0.2 -> joint=SFB1__SFP1_1 multiplier=2.9 offset=0.6

File: configs/urdf/heri_II.xacro (robot description, xacro)
@@ -98,5 +98,5 @@
     <child link="SFB1_1" />
     <axis xyz="0 0 -1" />
-    <limit lower="-0.1" upper="0.9" effort="10" velocity="1" />
+    <limit lower="-0.1" upper="0.2" effort="10" velocity="1" />
     <dynamics damping="0.003" friction="0.003"/>
   </joint>
@@ -132,9 +132,9 @@
     <limit lower="-0.1" upper="1.2" effort="10" velocity="1" />
     <dynamics damping="0.003" friction="0.003"/>
-    <mimic joint="SFB1__SFP1_1" multiplier="1.2" offset="0.2"/>
+    <mimic joint="SFB1__SFP1_1" multiplier="2.9" offset="0.6"/>
   </joint>
       <xacro:mimic_joint_plugin_gazebo name_prefix="SFP1_1__SFP1_2_joint"
     parent_joint="SFB1__SFP1_1" mimic_joint="SFP1_1__SFP1_2"
-    has_pid="false" multiplier="1.2" max_effort="10.0" offset="0.2"/>
+    has_pid="false" multiplier="2.9" max_effort="10.0" offset="0.6"/>
 <!-- ///////////////////////////////////////   Long finger 1   ////////////////////////////////////////// -->
   <!-- ///////////////////////////////////////   Base_Link of the long_finger   ////////////////////////////////////////// -->

Commit message: moving heri hal in other repo. one file still needed to be moved

File: configs/urdf/heri_II.urdf (robot description, URDF)
Before this commit: robot heri_II, 17 links, 16 joints
Links:
- added link LFP1_3_tip, mass 0.01
- added link LFP2_3_tip, mass 0.01
- added link LFP3_3_tip, mass 0.01
- added link SFP1_2_tip, mass 0.01
- added link motor_finger1_virtual_link, mass 0.01
- added link motor_finger2_virtual_link, mass 0.01
- added link motor_finger3_virtual_link, mass 0.01
- added link motor_thumb_virtual_link, mass 0.01
- link LFB1: geometry collision mesh filename=package://iit_heri_ii_hand_description/description/meshes/h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; visual mesh filename=package://iit_heri_ii_hand_description/description/meshes/h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
- link LFB2: geometry collision mesh filename=package://iit_heri_ii_hand_description/description/meshes/h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; visual mesh filename=package://iit_heri_ii_hand_description/description/meshes/h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
- link LFB3: geometry collision mesh filename=package://iit_heri_ii_hand_description/description/meshes/h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; visual mesh filename=package://iit_heri_ii_hand_description/description/meshes/h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
- link LFP1_1: geometry collision mesh filename=package://iit_heri_ii_hand_description/description/meshes/h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; visual mesh filename=package://iit_heri_ii_hand_description/description/meshes/h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
- link LFP1_2: geometry collision mesh filename=package://iit_heri_ii_hand_description/description/meshes/h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; visual mesh filename=package://iit_heri_ii_hand_description/description/meshes/h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
- link LFP1_3: geometry collision mesh filename=package://iit_heri_ii_hand_description/description/meshes/h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; visual mesh filename=package://iit_heri_ii_hand_description/description/meshes/h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
- link LFP2_1: geometry collision mesh filename=package://iit_heri_ii_hand_description/description/meshes/h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; visual mesh filename=package://iit_heri_ii_hand_description/description/meshes/h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
- link LFP2_2: geometry collision mesh filename=package://iit_heri_ii_hand_description/description/meshes/h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; visual mesh filename=package://iit_heri_ii_hand_description/description/meshes/h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
- link LFP2_3: geometry collision mesh filename=package://iit_heri_ii_hand_description/description/meshes/h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; visual mesh filename=package://iit_heri_ii_hand_description/description/meshes/h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
- link LFP3_1: geometry collision mesh filename=package://iit_heri_ii_hand_description/description/meshes/h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; visual mesh filename=package://iit_heri_ii_hand_description/description/meshes/h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
- link LFP3_2: geometry collision mesh filename=package://iit_heri_ii_hand_description/description/meshes/h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; visual mesh filename=package://iit_heri_ii_hand_description/description/meshes/h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
- link LFP3_3: geometry collision mesh filename=package://iit_heri_ii_hand_description/description/meshes/h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; visual mesh filename=package://iit_heri_ii_hand_description/description/meshes/h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
- link SFB1: geometry collision mesh filename=package://iit_heri_ii_hand_description/description/meshes/h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; visual mesh filename=package://iit_heri_ii_hand_description/description/meshes/h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
- link SFB1_1: geometry collision mesh filename=package://iit_heri_ii_hand_description/description/meshes/h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; visual mesh filename=package://iit_heri_ii_hand_description/description/meshes/h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
- link SFP1_2: geometry collision mesh filename=package://iit_heri_ii_hand_description/description/meshes/h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; visual mesh filename=package://iit_heri_ii_hand_description/description/meshes/h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
- link base_link: geometry collision mesh filename=package://iit_heri_ii_hand_description/description/meshes/h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; visual mesh filename=package://iit_heri_ii_hand_description/description/meshes/h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
Joints:
- added joint LFP1_3__LFP1_3_tip: type fixed, parent LFP1_3, child LFP1_3_tip, origin xyz=0.0175 -0.0111 0 rpy=1.5708 0 -0.13, axis 0 0 0
- added joint LFP2_3__LFP2_3_tip: type fixed, parent LFP2_3, child LFP2_3_tip, origin xyz=0.0175 -0.0111 0 rpy=1.5708 0 -0.13, axis 0 0 0
- added joint LFP3_3__LFP3_3_tip: type fixed, parent LFP3_3, child LFP3_3_tip, origin xyz=0.0175 -0.0111 0 rpy=1.5708 0 -0.13, axis 0 0 0
- added joint SFP1_2__SFP1_2_tip: type fixed, parent SFP1_2, child SFP1_2_tip, origin xyz=0.0175 -0.0111 0 rpy=1.5708 0 -0.13, axis 0 0 0
- added joint motor_finger1: type revolute, parent base_link, child motor_finger1_virtual_link, origin xyz=0 0 0 rpy=0 0 0, limit lower=0 upper=2.5 effort=10 velocity=1
- added joint motor_finger2: type revolute, parent base_link, child motor_finger2_virtual_link, origin xyz=0 0 0 rpy=0 0 0, limit lower=0 upper=2.5 effort=10 velocity=1
- added joint motor_finger3: type revolute, parent base_link, child motor_finger3_virtual_link, origin xyz=0 0 0 rpy=0 0 0, limit lower=0 upper=2.5 effort=10 velocity=1
- added joint motor_thumb: type revolute, parent base_link, child motor_thumb_virtual_link, origin xyz=7.6421E-05 -0.031634 0.1213 rpy=1.5708 -1.5708 0, limit lower=0 upper=2 effort=10 velocity=1
- joint LFB1__LFP1_1: limit lower=-0.1 upper=0.9 effort=10 velocity=1 -> lower=-0.1 upper=0.56 effort=10 velocity=1; mimic (none) -> joint=motor_finger1
- joint LFB2__LFP2_1: limit lower=-0.1 upper=0.73 effort=10 velocity=1 -> lower=-0.1 upper=0.56 effort=10 velocity=1; mimic (none) -> joint=motor_finger2
- joint LFB3__LFP3_1: limit lower=-0.1 upper=0.9 effort=10 velocity=1 -> lower=-0.1 upper=0.56 effort=10 velocity=1; mimic (none) -> joint=motor_finger3
- joint LFP1_1__LFP1_2: limit lower=-0.1 upper=0.5 effort=10 velocity=1 -> lower=-0.1 upper=1.22 effort=10 velocity=1; mimic joint=LFB1__LFP1_1 multiplier=1 offset=0.1 -> joint=motor_finger1
- joint LFP1_2__LFP1_3: limit lower=-0.1 upper=0.5 effort=10 velocity=1 -> lower=-0.1 upper=1.22 effort=10 velocity=1; mimic joint=LFB1__LFP1_1 multiplier=0.5 offset=0.2 -> joint=motor_finger1
- joint LFP2_1__LFP2_2: limit lower=-0.1 upper=0.5 effort=10 velocity=1 -> lower=-0.1 upper=1.22 effort=10 velocity=1; mimic joint=LFB2__LFP2_1 multiplier=1 offset=0.1 -> joint=motor_finger2
- joint LFP2_2__LFP2_3: limit lower=-0.1 upper=0.5 effort=10 velocity=1 -> lower=-0.1 upper=1.22 effort=10 velocity=1; mimic joint=LFB2__LFP2_1 multiplier=0.5 offset=0.2 -> joint=motor_finger2
- joint LFP3_1__LFP3_2: limit lower=-0.1 upper=0.5 effort=10 velocity=1 -> lower=-0.1 upper=1.22 effort=10 velocity=1; mimic joint=LFB3__LFP3_1 multiplier=1 offset=0.1 -> joint=motor_finger3
- joint LFP3_2__LFP3_3: limit lower=-0.1 upper=0.5 effort=10 velocity=1 -> lower=-0.1 upper=1.22 effort=10 velocity=1; mimic joint=LFB3__LFP3_1 multiplier=0.5 offset=0.2 -> joint=motor_finger3
- joint SFB1__SFP1_1: limit lower=-0.1 upper=0.9 effort=10 velocity=1 -> lower=-0.1 upper=1.22 effort=10 velocity=1; mimic (none) -> joint=motor_thumb; origin xyz=0.011 0 0.007 rpy=1.5708 -0.29671 0 -> xyz=0.0211 0 0.007 rpy=1.5708 -0.29671 0
- joint SFP1_1__SFP1_2: limit lower=-0.1 upper=1.2 effort=10 velocity=1 -> lower=-0.1 upper=1.22 effort=10 velocity=1; mimic joint=SFB1__SFP1_1 multiplier=1.2 offset=0.2 -> joint=motor_thumb

Commit message: modifications for exp with inail arm

File: configs/urdf/heri_II.urdf (robot description, URDF)
Before this commit: robot heri_II, 25 links, 24 joints
Joints:
- joint motor_finger1: limit lower=0 upper=2.5 effort=10 velocity=1 -> lower=-0.1 upper=2.51 effort=10 velocity=1
- joint motor_finger2: limit lower=0 upper=2.5 effort=10 velocity=1 -> lower=-0.1 upper=2.51 effort=10 velocity=1
- joint motor_finger3: limit lower=0 upper=2.5 effort=10 velocity=1 -> lower=-0.1 upper=2.51 effort=10 velocity=1
- joint motor_thumb: limit lower=0 upper=2 effort=10 velocity=1 -> lower=-0.1 upper=1.71 effort=10 velocity=1
