Commit message: model softhand updated

File: configs/urdf/qbhand.urdf (robot description, URDF)
Before this commit: robot qbhand, 38 links, 37 joints
Links:
- removed link qbhand_tendon_virtual_link
- added link qbhand_end_effector_link
- added link qbhand_synergy_tendon_virtual_link, mass 1e-4
- link qbhand_base_link: mass 0.15 -> 0.45
- link qbhand_index_distal_link: mass 0.01 -> 0.009; geometry collision mesh filename=package://qb_hand_description/meshes/ph_distal_collision.stl scale=0.001 0.001 0.001; visual mesh filename=package://qb_hand_description/meshes/ph_distal.stl scale=0.001 0.001 0.001
- link qbhand_index_distal_virtual_link: mass 0.01 -> 1e-4
- link qbhand_index_knuckle_link: mass 0.01 -> 0.0095; geometry collision mesh filename=package://qb_hand_description/meshes/ph_knuckle_collision.s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 scale=0.001 0.001 0.001; visual mesh filename=package://qb_hand_description/meshes/ph_knuckle.stl scale=0.001 0.001 0.001
- link qbhand_index_middle_link: mass 0.01 -> 0.0063
- link qbhand_index_middle_virtual_link: mass 0.01 -> 1e-4
- link qbhand_index_proximal_link: mass 0.01 -> 0.0082; geometry collision mesh filename=package://qb_hand_description/meshes/ph_medium_collision.stl scale=0.001 0.001 0.001; visual mesh filename=package://qb_hand_description/meshes/ph_medium.stl scale=0.001 0.001 0.001
- link qbhand_index_proximal_virtual_link: mass 0.01 -> 1e-4
- link qbhand_little_distal_link: mass 0.01 -> 0.009; geometry collision mesh filename=package://qb_hand_description/meshes/ph_distal_collision.stl scale=0.001 0.001 0.001; visual mesh filename=package://qb_hand_description/meshes/ph_distal.stl scale=0.001 0.001 0.001
- link qbhand_little_distal_virtual_link: mass 0.01 -> 1e-4
- link qbhand_little_knuckle_link: mass 0.01 -> 0.0095; geometry collision mesh filename=package://qb_hand_description/meshes/ph_knuckle_collision.s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 scale=0.001 0.001 0.001; visual mesh filename=package://qb_hand_description/meshes/ph_knuckle.stl scale=0.001 0.001 0.001
- link qbhand_little_middle_link: mass 0.01 -> 0.0063
- link qbhand_little_middle_virtual_link: mass 0.01 -> 1e-4
- link qbhand_little_proximal_link: mass 0.01 -> 0.0063
- link qbhand_little_proximal_virtual_link: mass 0.01 -> 1e-4
- link qbhand_middle_distal_link: mass 0.01 -> 0.009; geometry collision mesh filename=package://qb_hand_description/meshes/ph_distal_collision.stl scale=0.001 0.001 0.001; visual mesh filename=package://qb_hand_description/meshes/ph_distal.stl scale=0.001 0.001 0.001
- link qbhand_middle_distal_virtual_link: mass 0.01 -> 1e-4
- link qbhand_middle_knuckle_link: mass 0.01 -> 0.0095; geometry collision mesh filename=package://qb_hand_description/meshes/ph_knuckle_collision.s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 scale=0.001 0.001 0.001; visual mesh filename=package://qb_hand_description/meshes/ph_knuckle.stl scale=0.001 0.001 0.001
- link qbhand_middle_middle_link: mass 0.01 -> 0.0063
- link qbhand_middle_middle_virtual_link: mass 0.01 -> 1e-4
- link qbhand_middle_proximal_link: mass 0.01 -> 0.0082; geometry collision mesh filename=package://qb_hand_description/meshes/ph_medium_collision.stl scale=0.001 0.001 0.001; visual mesh filename=package://qb_hand_description/meshes/ph_medium.stl scale=0.001 0.001 0.001
- link qbhand_middle_proximal_virtual_link: mass 0.01 -> 1e-4
- link qbhand_palm_link: mass 0.36 -> 0.45
- link qbhand_ring_distal_link: mass 0.01 -> 0.009; geometry collision mesh filename=package://qb_hand_description/meshes/ph_distal_collision.stl scale=0.001 0.001 0.001; visual mesh filename=package://qb_hand_description/meshes/ph_distal.stl scale=0.001 0.001 0.001
- link qbhand_ring_distal_virtual_link: mass 0.01 -> 1e-4
- link qbhand_ring_knuckle_link: mass 0.01 -> 0.0095; geometry collision mesh filename=package://qb_hand_description/meshes/ph_knuckle_collision.s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 scale=0.001 0.001 0.001; visual mesh filename=package://qb_hand_description/meshes/ph_knuckle.stl scale=0.001 0.001 0.001
- link qbhand_ring_middle_link: mass 0.01 -> 0.0063
- link qbhand_ring_middle_virtual_link: mass 0.01 -> 1e-4
- link qbhand_ring_proximal_link: mass 0.01 -> 0.0082; geometry collision mesh filename=package://qb_hand_description/meshes/ph_medium_collision.stl scale=0.001 0.001 0.001; visual mesh filename=package://qb_hand_description/meshes/ph_medium.stl scale=0.001 0.001 0.001
- link qbhand_ring_proximal_virtual_link: mass 0.01 -> 1e-4
- link qbhand_thumb_distal_link: mass 0.01 -> 0.009; geometry collision mesh filename=package://qb_hand_description/meshes/ph_distal_collision.stl scale=0.001 0.001 0.001; visual mesh filename=package://qb_hand_description/meshes/ph_distal.stl scale=0.001 0.001 0.001
- link qbhand_thumb_distal_virtual_link: mass 0.01 -> 1e-4
- link qbhand_thumb_knuckle_link: geometry collision mesh filename=package://qb_hand_description/meshes/ph_thumb_r_collision.s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 scale=0.001 0.001 0.001; visual mesh filename=package://qb_hand_description/meshes/ph_thumb_r.stl scale=0.001 0.001 0.001
- link qbhand_thumb_proximal_link: mass 0.01 -> 0.0063
- link qbhand_thumb_proximal_virtual_link: mass 0.01 -> 1e-4
Joints:
- added joint qbhand_end_effector_fixed_joint: type fixed, parent qbhand_base_link, child qbhand_end_effector_link, origin xyz=-0.03 0.060 0.142 rpy=-1.57 0 0
- joint qbhand_index_knuckle_joint: origin xyz=-0.02 -0.007 0.014 rpy=0 0 0 -> xyz=-0.02 -0.007 0.014 rpy=0 0 1.57
- joint qbhand_index_proximal_joint: origin xyz=0 0.009 0 rpy=1.57 0 1.57 -> xyz=0.009 0 0 rpy=1.57 0 0
- joint qbhand_little_knuckle_joint: origin xyz=0.04 -0.012 0.014 rpy=0 0 0 -> xyz=0.04 -0.012 0.014 rpy=0 0 1.57
- joint qbhand_little_proximal_joint: origin xyz=0 0.009 0 rpy=1.57 0 1.57 -> xyz=0.009 0 0 rpy=1.57 0 0
- joint qbhand_middle_knuckle_joint: origin xyz=0 0 0.014 rpy=0 0 0 -> xyz=0 0 0.014 rpy=0 0 1.57
- joint qbhand_middle_proximal_joint: origin xyz=0 0.009 0 rpy=1.57 0 1.57 -> xyz=0.009 0 0 rpy=1.57 0 0
- joint qbhand_ring_knuckle_joint: origin xyz=0.02 -0.007 0.014 rpy=0 0 0 -> xyz=0.02 -0.007 0.014 rpy=0 0 1.57
- joint qbhand_ring_proximal_joint: origin xyz=0 0.009 0 rpy=1.57 0 1.57 -> xyz=0.009 0 0 rpy=1.57 0 0
- joint qbhand_synergy_joint: child qbhand_tendon_virtual_link -> qbhand_synergy_tendon_virtual_link
- joint qbhand_thumb_knuckle_joint: origin xyz=-0.0435 -0.0435 -0.002 rpy=-1.57 3.14 0 -> xyz=-0.044 -0.0465 -0.002 rpy=-1.57 3.14 0.0
- joint qbhand_thumb_proximal_joint: origin xyz=0.0255 -0.004 -0.0025 rpy=-1.15 0.0 0.0 -> xyz=0.0255 -0.0038 -0.00012 rpy=-1.1415 0.0 0.0
