Commit message: updated model

File: configs/urdf/onrobot_3fg15.urdf (robot description, URDF)
Before this commit: robot onrobot_3fg15, 5 links, 4 joints
Joints:
- joint robot_onrobot_3fg15_finger_joint1: limit lower=0.0 upper=2.8 effort=20 velocity=3.0 -> lower=0.0 upper=2.9 effort=20 velocity=3.0
- joint robot_onrobot_3fg15_finger_joint2: limit lower=0.0 upper=2.8 effort=20 velocity=3.0 -> lower=0.0 upper=2.9 effort=20 velocity=3.0
- joint robot_onrobot_3fg15_finger_joint3: limit lower=0.0 upper=2.8 effort=20 velocity=3.0 -> lower=0.0 upper=2.9 effort=20 velocity=3.0

Commit message: better (less wrong) onrobot 3fg15 inertia values

File: configs/urdf/onrobot_3fg15.urdf (robot description, URDF)
Before this commit: robot onrobot_3fg15, 5 links, 4 joints
Links:
- link robot_onrobot_3fg15_base_link: mass 0.54 -> 1.15
