Commit message: dagana final fixes

File: configs/urdf/dagana.urdf (robot description, URDF)
Before this commit: robot dagana, 4 links, 3 joints
Joints:
- joint dagana_gripper_claw_joint: axis -1 0 0 -> 1 0 0; origin xyz=0.0 -0.028 0.05025 rpy=1.57079632679 0 3.14159265359 -> xyz=0.0 -0.028 0.05025 rpy=0.5 0 3.14159265359
